File: ArmazCape/Rev B1/ArmazCape - Rev B1.brd (EAGLE design)
At the start: 85 x 70.5 mm, 135 parts, among them Q1 32.768kHz, 12.5pF, Q2 16MHz, 22pF, Q4 IRLML6344TRPBF, Q5 IRLML6344TRPBF, U1 L7985A, U10 MCP2515-I/SO, U12 24AA256-I/SN, U13 L7985A, U2 SN65HVD232D, U4 DS1307ZN+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

Commit message: Last update of ArmazCape - Rev B1 We know focus on Rev B2
Connections:
- new net MCP2515_INT: BB1.P9.27, U10.12
Routing:
- net MCP2515_INT: track 0.00 -> 38.2 mm, vias 0 -> 1
Changed lines of the file:
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@@
 <wire x1="28.575" y1="32.004" x2="31.75" y2="32.004" width="0.1778" layer="1"/>
 <wire x1="31.75" y1="32.004" x2="34.544" y2="34.798" width="0.1778" layer="1"/>
-<wire x1="34.544" y1="34.798" x2="34.544" y2="38.608" width="0.1778" layer="1"/>
-<wire x1="34.544" y1="38.608" x2="36.83" y2="40.894" width="0.1778" layer="1"/>
-<wire x1="36.83" y1="40.894" x2="37.338" y2="40.894" width="0.1778" layer="1"/>
-<wire x1="37.338" y1="40.894" x2="39.37" y2="42.926" width="0.1778" layer="1"/>
-<wire x1="39.37" y1="42.926" x2="39.37" y2="58.42" width="0.1778" layer="1"/>
+<wire x1="34.544" y1="34.798" x2="34.544" y2="37.1348" width="0.1778" layer="1"/>
+<wire x1="34.544" y1="37.1348" x2="36.83" y2="39.4208" width="0.1778" layer="1"/>
+<wire x1="36.83" y1="39.4208" x2="37.338" y2="39.4208" width="0.1778" layer="1"/>
+<wire x1="37.338" y1="39.4208" x2="39.37" y2="41.4528" width="0.1778" layer="1"/>
+<wire x1="39.37" y1="41.4528" x2="39.37" y2="58.42" width="0.1778" layer="1"/>
 <wire x1="39.37" y1="58.42" x2="38.862" y2="58.928" width="0.1778" layer="1"/>
 </signal>
@@
 <wire x1="28.575" y1="30.734" x2="31.242" y2="30.734" width="0.1778" layer="1"/>
 <wire x1="31.242" y1="30.734" x2="35.052" y2="34.544" width="0.1778" layer="1"/>
-<wire x1="35.052" y1="34.544" x2="35.052" y2="38.354" width="0.1778" layer="1"/>
-<wire x1="35.052" y1="38.354" x2="37.084" y2="40.386" width="0.1778" layer="1"/>
-<wire x1="37.084" y1="40.386" x2="37.592" y2="40.386" width="0.1778" layer="1"/>
-<wire x1="37.592" y1="40.386" x2="39.878" y2="42.672" width="0.1778" layer="1"/>
-<wire x1="39.878" y1="42.672" x2="39.878" y2="58.166" width="0.1778" layer="1"/>
+<wire x1="35.052" y1="34.544" x2="35.052" y2="36.8808" width="0.1778" layer="1"/>
+<wire x1="35.052" y1="36.8808" x2="37.084" y2="38.9128" width="0.1778" layer="1"/>
+<wire x1="37.084" y1="38.9128" x2="37.592" y2="38.9128" width="0.1778" layer="1"/>
+<wire x1="37.592" y1="38.9128" x2="39.878" y2="41.1988" width="0.1778" layer="1"/>
+<wire x1="39.878" y1="41.1988" x2="39.878" y2="58.166" width="0.1778" layer="1"/>
 </signal>
 <signal name="SYS_5V" class="1">
@@
 <wire x1="28.575" y1="28.194" x2="30.226" y2="28.194" width="0.1778" layer="1"/>
 <wire x1="30.226" y1="28.194" x2="36.068" y2="34.036" width="0.1778" layer="1"/>
-<wire x1="36.068" y1="34.036" x2="36.068" y2="37.846" width="0.1778" layer="1"/>
-<wire x1="36.068" y1="37.846" x2="37.592" y2="39.37" width="0.1778" layer="1"/>
-<wire x1="37.592" y1="39.37" x2="38.1" y2="39.37" width="0.1778" layer="1"/>
-<wire x1="38.1" y1="39.37" x2="40.894" y2="42.164" width="0.1778" layer="1"/>
-<wire x1="40.894" y1="42.164" x2="40.894" y2="57.658" width="0.1778" layer="1"/>
+<wire x1="36.068" y1="34.036" x2="36.068" y2="36.3728" width="0.1778" layer="1"/>
+<wire x1="36.068" y1="36.3728" x2="37.592" y2="37.8968" width="0.1778" layer="1"/>
+<wire x1="37.592" y1="37.8968" x2="38.1" y2="37.8968" width="0.1778" layer="1"/>
+<wire x1="38.1" y1="37.8968" x2="40.894" y2="40.6908" width="0.1778" layer="1"/>
+<wire x1="40.894" y1="40.6908" x2="40.894" y2="57.658" width="0.1778" layer="1"/>
 </signal>
 <signal name="SPI1_MISO">
@@
 <wire x1="28.575" y1="29.464" x2="30.734" y2="29.464" width="0.1778" layer="1"/>
 <wire x1="30.734" y1="29.464" x2="35.56" y2="34.29" width="0.1778" layer="1"/>
-<wire x1="35.56" y1="34.29" x2="35.56" y2="38.1" width="0.1778" layer="1"/>
-<wire x1="35.56" y1="38.1" x2="37.338" y2="39.878" width="0.1778" layer="1"/>
-<wire x1="37.338" y1="39.878" x2="37.846" y2="39.878" width="0.1778" layer="1"/>
-<wire x1="37.846" y1="39.878" x2="40.386" y2="42.418" width="0.1778" layer="1"/>
-<wire x1="40.386" y1="42.418" x2="40.386" y2="57.912" width="0.1778" layer="1"/>
+<wire x1="35.56" y1="34.29" x2="35.56" y2="36.6268" width="0.1778" layer="1"/>
+<wire x1="35.56" y1="36.6268" x2="37.338" y2="38.4048" width="0.1778" layer="1"/>
+<wire x1="37.338" y1="38.4048" x2="37.846" y2="38.4048" width="0.1778" layer="1"/>
+<wire x1="37.846" y1="38.4048" x2="40.386" y2="40.9448" width="0.1778" layer="1"/>
+<wire x1="40.386" y1="40.9448" x2="40.386" y2="57.912" width="0.1778" layer="1"/>
 </signal>
 <signal name="VDD_ADC">
@@
 <wire x1="28.575" y1="26.924" x2="29.718" y2="26.924" width="0.1778" layer="1"/>
 <wire x1="29.718" y1="26.924" x2="36.576" y2="33.782" width="0.1778" layer="1"/>
-<wire x1="36.576" y1="33.782" x2="36.576" y2="37.592" width="0.1778" layer="1"/>
-<wire x1="36.576" y1="37.592" x2="37.846" y2="38.862" width="0.1778" layer="1"/>
-<wire x1="37.846" y1="38.862" x2="38.354" y2="38.862" width="0.1778" layer="1"/>
-<wire x1="38.354" y1="38.862" x2="41.402" y2="41.91" width="0.1778" layer="1"/>
-<wire x1="41.402" y1="41.91" x2="41.402" y2="54.61" width="0.1778" layer="1"/>
+<wire x1="36.576" y1="33.782" x2="36.576" y2="36.1188" width="0.1778" layer="1"/>
+<wire x1="36.576" y1="36.1188" x2="37.846" y2="37.3888" width="0.1778" layer="1"/>
+<wire x1="37.846" y1="37.3888" x2="38.354" y2="37.3888" width="0.1778" layer="1"/>
+<wire x1="38.354" y1="37.3888" x2="41.402" y2="40.4368" width="0.1778" layer="1"/>
+<wire x1="41.402" y1="40.4368" x2="41.402" y2="54.61" width="0.1778" layer="1"/>
 <wire x1="41.402" y1="54.61" x2="41.91" y2="55.118" width="0.1778" layer="1"/>
 <via x="41.91" y="55.118" extent="1-16" drill="0.35"/>
@@
 <wire x1="11.596" y1="48.514" x2="9.994" y2="48.514" width="0.3048" layer="1"/>
 </signal>
+<signal name="MCP2515_INT">
+<contactref element="BB1" pad="P9.27"/>
+<contactref element="U10" pad="12"/>
+<wire x1="28.575" y1="33.274" x2="32.258" y2="33.274" width="0.1778" layer="1"/>
+<wire x1="32.258" y1="33.274" x2="34.036" y2="35.052" width="0.1778" layer="1"/>
+<wire x1="34.036" y1="35.052" x2="34.036" y2="37.3888" width="0.1778" layer="1"/>
+<wire x1="34.036" y1="37.3888" x2="36.576" y2="39.9288" width="0.1778" layer="1"/>
+<wire x1="36.576" y1="39.9288" x2="37.084" y2="39.9288" width="0.1778" layer="1"/>
+<wire x1="37.084" y1="39.9288" x2="38.862" y2="41.7068" width="0.1778" layer="1"/>
+<wire x1="38.862" y1="41.7068" x2="38.862" y2="57.658" width="0.1778" layer="1"/>
+<wire x1="38.862" y1="57.658" x2="38.608" y2="57.912" width="0.1778" layer="1"/>
+<via x="38.608" y="57.912" extent="1-16" drill="0.35"/>
+<wire x1="38.608" y1="57.912" x2="38.862" y2="58.166" width="0.1778" layer="16"/>
+<wire x1="38.862" y1="58.166" x2="38.862" y2="59.944" width="0.1778" layer="16"/>
+<wire x1="38.862" y1="59.944" x2="39.624" y2="60.706" width="0.1778" layer="16"/>
+<wire x1="39.624" y1="60.706" x2="41.402" y2="60.706" width="0.1778" layer="16"/>
+<wire x1="41.402" y1="60.706" x2="42.672" y2="61.976" width="0.1778" layer="16"/>
+</signal>
 </signals>
