File: ArmazConnect/Rev B1/ArmazConnect - Rev B1.sch (EAGLE design)
At the start: 40 parts, among them X0 NC3FAAV2, X1 NC3FAAV2, X2 NC3FAAV2, X3 NC3FAAV2, X4 NC5FAV-SW, X5 NC5MAV-SW, X6 NC5FAV-SW, X7 5504F1-09S-02A-03, X8 87832-26

Commit message: Latest changes on ArmazConnect - Rev B1
Parts:
- C1, C2: MPN MC0805B561K500CT -> MC0603B561K500CT; OC_FARNELL 1759219 -> 1759081
- C3: MPN MC0805F105Z250CT -> MC0603F105Z250CT; OC_FARNELL 1759429 -> 1759039
- C4, C5: MPN MC0805F105Z250CT -> MC0805F105Z500CT; OC_FARNELL 1759429 -> 1759432
- R0, R1, R2, R3, R4: MPN MCMR04X1501FTL -> MCMR06X1501FTL; OC_FARNELL 2072645 -> 2073391
- R24: MPN MC00625W040213K3 -> MCMR04X3301FTL; OC_FARNELL 1358056 -> 2072928
- R25: MPN MC00625W04021330R -> MCMR04X3300FTL; OC_FARNELL 1358028 -> 2072927
- R26, R27: MPN MC00625W040214K7 -> MCMR06X4701FTL; OC_FARNELL 1358060 -> 2073509
- R5, R6: MPN MC00625W04021100R -> MCMR06X1000FTL; OC_FARNELL 1358015 -> 2073347
- R7: MPN MC00625W04021120R -> MCMR06X1200FTL; OC_FARNELL 1358018 -> 2073369
Connections:
- net +12V: now also X7C.9; no longer X7.9
- net CAN0-H: now also X7C.7; no longer X7.7
- net CAN0-L: now also X7C.2; no longer X7.2
- net CAN0_GND: now also X7C.3, X7C.6; no longer X7.3, X7.6
- net CAN0_SHIELD: now also X7C.5; no longer X7.5
- net GND1: now also X7S.SHIELD
Changed lines of the file:
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@@
 <part name="R0" library="rcl" deviceset="R-EU_" device="R0603" value="1.5K">
 <attribute name="MF" value="MULTICOMP"/>
-<attribute name="MPN" value="MCMR04X1501FTL"/>
-<attribute name="OC_FARNELL" value="2072645"/>
+<attribute name="MPN" value="MCMR06X1501FTL"/>
+<attribute name="OC_FARNELL" value="2073391"/>
 </part>
 <part name="LED0" library="led" deviceset="LED" device="CHIP-LED0603" value="blue">
@@
 <part name="R1" library="rcl" deviceset="R-EU_" device="R0603" value="1.5K">
 <attribute name="MF" value="MULTICOMP"/>
-<attribute name="MPN" value="MCMR04X1501FTL"/>
-<attribute name="OC_FARNELL" value="2072645"/>
+<attribute name="MPN" value="MCMR06X1501FTL"/>
+<attribute name="OC_FARNELL" value="2073391"/>
 </part>
 <part name="LED1" library="led" deviceset="LED" device="CHIP-LED0603" value="blue">
@@
 <part name="R2" library="rcl" deviceset="R-EU_" device="R0603" value="1.5K">
 <attribute name="MF" value="MULTICOMP"/>
-<attribute name="MPN" value="MCMR04X1501FTL"/>
-<attribute name="OC_FARNELL" value="2072645"/>
+<attribute name="MPN" value="MCMR06X1501FTL"/>
+<attribute name="OC_FARNELL" value="2073391"/>
 </part>
 <part name="LED2" library="led" deviceset="LED" device="CHIP-LED0603" value="blue">
@@
 <part name="R3" library="rcl" deviceset="R-EU_" device="R0603" value="1.5K">
 <attribute name="MF" value="MULTICOMP"/>
-<attribute name="MPN" value="MCMR04X1501FTL"/>
-<attribute name="OC_FARNELL" value="2072645"/>
+<attribute name="MPN" value="MCMR06X1501FTL"/>
+<attribute name="OC_FARNELL" value="2073391"/>
 </part>
 <part name="LED3" library="led" deviceset="LED" device="CHIP-LED0603" value="blue">
@@
 <part name="R4" library="rcl" deviceset="R-EU_" device="R0603" value="1.5K">
 <attribute name="MF" value="MULTICOMP"/>
-<attribute name="MPN" value="MCMR04X1501FTL"/>
-<attribute name="OC_FARNELL" value="2072645"/>
+<attribute name="MPN" value="MCMR06X1501FTL"/>
+<attribute name="OC_FARNELL" value="2073391"/>
 </part>
 <part name="LED4" library="led" deviceset="LED" device="CHIP-LED0603" value="blue">
@@
 <part name="R5" library="rcl" deviceset="R-EU_" device="R0603" value="100">
 <attribute name="MF" value="MULTICOMP"/>
-<attribute name="MPN" value="MC00625W04021100R"/>
-<attribute name="OC_FARNELL" value="1358015"/>
+<attribute name="MPN" value="MCMR06X1000FTL"/>
+<attribute name="OC_FARNELL" value="2073347"/>
 </part>
 <part name="R6" library="rcl" deviceset="R-EU_" device="R0603" value="100">
 <attribute name="MF" value="MULTICOMP"/>
-<attribute name="MPN" value="MC00625W04021100R"/>
-<attribute name="OC_FARNELL" value="1358015"/>
+<attribute name="MPN" value="MCMR06X1000FTL"/>
+<attribute name="OC_FARNELL" value="2073347"/>
 </part>
 <part name="C1" library="rcl" deviceset="C-EU" device="C0603" value="560pF">
 <attribute name="MF" value="MULTICOMP"/>
-<attribute name="MPN" value="MC0805B561K500CT"/>
-<attribute name="OC_FARNELL" value="1759219"/>
+<attribute name="MPN" value="MC0603B561K500CT"/>
+<attribute name="OC_FARNELL" value="1759081"/>
 </part>
 <part name="C2" library="rcl" deviceset="C-EU" device="C0603" value="560pF">
 <attribute name="MF" value="MULTICOMP"/>
-<attribute name="MPN" value="MC0805B561K500CT"/>
-<attribute name="OC_FARNELL" value="1759219"/>
+<attribute name="MPN" value="MC0603B561K500CT"/>
+<attribute name="OC_FARNELL" value="1759081"/>
 </part>
 <part name="SUPPLY4" library="supply2" deviceset="+12V" device=""/>
 <part name="C3" library="rcl" deviceset="C-EU" device="C0603" value="1uF">
 <attribute name="MF" value="MULTICOMP"/>
-<attribute name="MPN" value="MC0805F105Z250CT"/>
-<attribute name="OC_FARNELL" value="1759429"/>
+<attribute name="MPN" value="MC0603F105Z250CT"/>
+<attribute name="OC_FARNELL" value="1759039"/>
 </part>
 <part name="SUPPLY5" library="supply2" deviceset="GND1" device=""/>
@@
 <part name="R7" library="rcl" deviceset="R-EU_" device="R0603" value="120">
 <attribute name="MF" value="MULTICOMP"/>
-<attribute name="MPN" value="MC00625W04021120R"/>
-<attribute name="OC_FARNELL" value="1358018"/>
+<attribute name="MPN" value="MCMR06X1200FTL"/>
+<attribute name="OC_FARNELL" value="2073369"/>
 </part>
 <part name="GND6" library="supply1" deviceset="GND" device=""/>
@@
 <part name="R24" library="rcl" deviceset="R-EU_" device="R0402" value="3K3">
 <attribute name="MF" value="MULTICOMP"/>
-<attribute name="MPN" value="MC00625W040213K3"/>
-<attribute name="OC_FARNELL" value="1358056"/>
+<attribute name="MPN" value="MCMR04X3301FTL"/>
+<attribute name="OC_FARNELL" value="2072928"/>
 </part>
 <part name="R25" library="rcl" deviceset="R-EU_" device="R0603" value="330">
 <attribute name="MF" value="MULTICOMP"/>
-<attribute name="MPN" value="MC00625W04021330R"/>
-<attribute name="OC_FARNELL" value="1358028"/>
+<attribute name="MPN" value="MCMR04X3300FTL"/>
+<attribute name="OC_FARNELL" value="2072927"/>
 </part>
 <part name="R26" library="rcl" deviceset="R-EU_" device="R0603" value="4K7">
 <attribute name="MF" value="MULTICOMP"/>
-<attribute name="MPN" value="MC00625W040214K7"/>
-<attribute name="OC_FARNELL" value="1358060"/>
+<attribute name="MPN" value="MCMR06X4701FTL"/>
+<attribute name="OC_FARNELL" value="2073509"/>
 </part>
 <part name="R27" library="rcl" deviceset="R-EU_" device="R0603" value="4K7">
 <attribute name="MF" value="MULTICOMP"/>
-<attribute name="MPN" value="MC00625W040214K7"/>
-<attribute name="OC_FARNELL" value="1358060"/>
+<attribute name="MPN" value="MCMR06X4701FTL"/>
+<attribute name="OC_FARNELL" value="2073509"/>
 </part>
 <part name="GND" library="wirepad" deviceset="WIREPAD" device="1,6/0,9" value="WIREPAD1,6/0,9">
@@
 <part name="C4" library="rcl" deviceset="C-EU" device="C0805" value="1uF">
 <attribute name="MF" value="MULTICOMP"/>
-<attribute name="MPN" value="MC0805F105Z250CT"/>
-<attribute name="OC_FARNELL" value="1759429"/>
+<attribute name="MPN" value="MC0805F105Z500CT"/>
+<attribute name="OC_FARNELL" value="1759432"/>
 </part>
 <part name="C5" library="rcl" deviceset="C-EU" device="C0805" value="1uF">
 <attribute name="MF" value="MULTICOMP"/>
-<attribute name="MPN" value="MC0805F105Z250CT"/>
-<attribute name="OC_FARNELL" value="1759429"/>
+<attribute name="MPN" value="MC0805F105Z500CT"/>
+<attribute name="OC_FARNELL" value="1759432"/>
 </part>
 <part name="P+3" library="supply1" deviceset="+5V" device=""/>
@@
 <part name="+3V2" library="supply1" deviceset="+3V3" device=""/>
 <part name="+3V3" library="supply1" deviceset="+3V3" device=""/>
+<part name="SUPPLY13" library="supply2" deviceset="GND1" device=""/>
 </parts>
 <sheets>
@@
 <instance part="X5" gate="-1" x="22.86" y="99.06" rot="MR0"/>
 <instance part="GND13" gate="1" x="38.1" y="144.78"/>
-<instance part="X7" gate="G$1" x="335.28" y="144.78">
+<instance part="X7" gate="C" x="335.28" y="144.78">
 <attribute name="OC_FARNELL" x="335.28" y="144.78" size="1.27" layer="96" display="off"/>
 <attribute name="MF" x="335.28" y="144.78" size="1.27" layer="96" display="off"/>
@@
 <instance part="+3V2" gate="G$1" x="129.54" y="144.78"/>
 <instance part="+3V3" gate="G$1" x="167.64" y="142.24"/>
+<instance part="X7" gate="S" x="330.2" y="119.38"/>
+<instance part="SUPPLY13" gate="G$1" x="330.2" y="109.22"/>
 </instances>
 <busses>
@@
 <net name="CAN0-L" class="0">
 <segment>
-<pinref part="X7" gate="G$1" pin="2"/>
+<pinref part="X7" gate="C" pin="2"/>
 <label x="325.12" y="147.32" size="1.27" layer="95" rot="MR0"/>
 <wire x1="327.66" y1="147.32" x2="307.34" y2="147.32" width="0.1524" layer="91"/>
@@
 <net name="CAN0-H" class="0">
 <segment>
-<pinref part="X7" gate="G$1" pin="7"/>
+<pinref part="X7" gate="C" pin="7"/>
 <label x="345.44" y="144.78" size="1.27" layer="95"/>
 <wire x1="342.9" y1="144.78" x2="363.22" y2="144.78" width="0.1524" layer="91"/>
@@
 <net name="+12V" class="1">
 <segment>
-<pinref part="X7" gate="G$1" pin="9"/>
+<pinref part="X7" gate="C" pin="9"/>
 <wire x1="342.9" y1="139.7" x2="347.98" y2="139.7" width="0.1524" layer="91"/>
 <label x="345.44" y="139.7" size="1.27" layer="95"/>
@@
 <pinref part="SUPPLY12" gate="G$1" pin="GND1"/>
 <wire x1="167.64" y1="127" x2="167.64" y2="129.54" width="0.1524" layer="91"/>
+</segment>
+<segment>
+<pinref part="X7" gate="S" pin="SHIELD"/>
+<pinref part="SUPPLY13" gate="G$1" pin="GND1"/>
+<wire x1="330.2" y1="111.76" x2="330.2" y2="116.84" width="0.1524" layer="91"/>
 </segment>
 </net>
@@
 <net name="CAN0_SHIELD" class="0">
 <segment>
-<pinref part="X7" gate="G$1" pin="5"/>
+<pinref part="X7" gate="C" pin="5"/>
 <wire x1="327.66" y1="139.7" x2="322.58" y2="139.7" width="0.1524" layer="91"/>
 <label x="325.12" y="139.7" size="1.27" layer="95" rot="MR0"/>
@@
 <net name="CAN0_GND" class="0">
 <segment>
-<pinref part="X7" gate="G$1" pin="3"/>
+<pinref part="X7" gate="C" pin="3"/>
 <label x="325.12" y="144.78" size="1.27" layer="95" rot="MR0"/>
 <wire x1="327.66" y1="144.78" x2="312.42" y2="144.78" width="0.1524" layer="91"/>
@@
 </segment>
 <segment>
-<pinref part="X7" gate="G$1" pin="6"/>
+<pinref part="X7" gate="C" pin="6"/>
 <label x="345.44" y="147.32" size="1.27" layer="95"/>
 <wire x1="342.9" y1="147.32" x2="358.14" y2="147.32" width="0.1524" layer="91"/>
