File: ArmazEthernet/Rev A1/ArmazEthernet- Rev A1.brd (EAGLE design)
At the start: 68 x 80 mm, 112 parts, among them M1:C1 1000pF, 2kV, M1:C2 .022uF, M1:C3 15pF, 50V, M1:C4 15pF, 50V, M1:C5 15pF, 50V, M1:C6 15pF, 50V, M1:R1 75, M1:R2 75, M1:R3 75, M1:R4 75, M1:R5 10, 1/8W, 1%, U1 LAN9303-ABZJ, U2 LAN8710AI-EZK, U3 LP2992IM5-3.3, X10 85505-5113, X8 87832-26

Commit message: Added missing lib: atmel.lbr Provides ATMega328
Parts:
- removed X8: 87832-26, con-molex:87832-26
- C23, C24, C25, C26: device rcl:C0402 -> rcl:C0603
- E0:M:C3, E0:M:C4, E0:M:C5, E0:M:C6, E1:M:C3, E1:M:C4, E1:M:C5, E1:M:C6, M1:C3, M1:C4, M1:C5, M1:C6: device rcl:C0504 -> rcl:C0603
- E0:M:R1, E0:M:R2, E0:M:R3, E0:M:R4, E0:M:R5, E1:M:R1, E1:M:R2, E1:M:R3, E1:M:R4, E1:M:R5, F0:R6, F0:R7, F0:R8, F0:R9, F1:R6, F1:R7, F1:R8, F1:R9, F2:R6, F2:R7, F2:R8, F2:R9, M1:R1, M1:R2, M1:R3, M1:R4, M1:R5, R10, R11, R12, R13, R14, R15, R16, R17, R18, R19, R20, R21, R22, SJ2, SJ3, SJ4, SJ5: device rcl:R0402 -> rcl:R0603
- moved SJ5 230.4 mm to (55.1, 43.2), turned to 270 degrees
- moved R17 228.0 mm to (54.4, 45.7), turned to 180 degrees
- moved SJ4 223.5 mm to (51.6, 43.2), turned to 270 degrees
- moved C29 221.9 mm to (46.7, 64.5), turned to 270 degrees
- moved C25 218.1 mm to (65.8, 68.8)
- moved SJ3 216.9 mm to (48.0, 43.2), turned to 270 degrees
- moved R16 216.3 mm to (55.1, 48.3), turned to 270 degrees
- moved C28 216.1 mm to (48.8, 64.5), turned to 270 degrees
- moved R11 215.6 mm to (44.5, 48.3), turned to 90 degrees
- moved C15 211.8 mm to (51.3, 57.4), turned to 90 degrees
- moved C17 211.4 mm to (37.8, 42.9), turned to 270 degrees
- moved SJ2 210.7 mm to (44.5, 43.2), turned to 270 degrees
- moved O1 207.1 mm to (20.3, 53.6), turned to 180 degrees
- moved R10 207.0 mm to (43.7, 45.7)
- moved R15 206.0 mm to (50.8, 45.7), turned to 180 degrees
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Connections:
- removed net +12V: X8.21, X8.22
- removed net +5V/1: X8.23
- removed net CAN0-H: X8.14
- removed net CAN0-L: X8.13
- removed net DMX0-A: X8.11
- removed net DMX0-B: X8.12
- removed net DV0: X8.15
- removed net ESW0: X8.5
- removed net ESW1: X8.6
- removed net ESW2: X8.7
- removed net ESW3: X8.8
- removed net FAN0_GND: X8.19
- removed net FAN1_GND: X8.20
- removed net GND1: X8.25, X8.26
- removed net UART5_RXD: X8.9
- removed net UART5_TXD: X8.10
- removed net VDD_3V3: X8.24
- net +5V: no longer X8.1, X8.2
- net GND: no longer X8.3, X8.4
Routing:
- net E0:M:N$1: track 0.00 -> 57.9 mm, vias 0 -> 1
- net N$22: track 0.00 -> 54.5 mm, vias 0 -> 3
- net N$24: track 0.00 -> 53.0 mm, vias 0 -> 3
- net N$25: track 0.00 -> 48.7 mm, vias 0 -> 1
- net N$300: track 0.00 -> 47.5 mm, vias 0 -> 2
- net N$301: track 0.00 -> 43.9 mm, vias 0 -> 3
- net E1:M:N$1: track 0.00 -> 43.6 mm, vias 0 -> 1
- net N$23: track 0.00 -> 42.3 mm, vias 0 -> 1
- net N$303: track 0.00 -> 35.3 mm, vias 0 -> 3
- net N$302: track 0.00 -> 32.1 mm
- net E1:N$5: track 0.00 -> 28.1 mm, vias 0 -> 2
- net E1:N$6: track 0.00 -> 23.3 mm, vias 0 -> 4
- net E0:N$5: track 0.00 -> 20.6 mm
- net E0:N$3: track 0.00 -> 20.0 mm
- net E0:M:N$3: track 0.00 -> 19.8 mm, vias 0 -> 1
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- added copper zone on layer 1, net +3V3
- added copper zone on layer 3, net +3V3
- added copper zone on layer 1, net +5V
- added copper zone on layer 1, net GND
- added copper zone on layer 16, net GND
- added copper zone on layer 2, net GND
