File: LED LAMP/VarmoLed - Rev A1.brd (EAGLE design)
At the start: 25 x 46 mm, 20 parts, among them J1 22-05-7038-03, U1 IRLML6344TRPBF

Commit message: Rename Varmo LED to lamp LED and add a resitor on input of the transistor
Parts:
- added R6: 100, rcl:R0603
Connections:
- new net N$6: R6.2, U1.1
- net LED_CMD: now also R6.1; no longer U1.1
Routing:
- net N$6: track 0.00 -> 2.42 mm
- net LED_CMD: track 8.84 -> 10.6 mm
Changed lines of the file:
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@@
 <setting verticaltext="up"/>
 </settings>
-<grid distance="1" unitdist="mm" unit="mil" style="dots" multiple="2" display="yes" altdistance="0.25" altunitdist="mm" altunit="mm"/>
+<grid distance="1" unitdist="mm" unit="mm" style="dots" multiple="2" display="yes" altdistance="0.25" altunitdist="mm" altunit="mm"/>
 <layers>
 <layer number="1" name="Top" color="4" fill="1" visible="yes" active="yes"/>
@@
 <attribute name="VALUE" x="10.2956" y="30.805" size="0.4064" layer="27" ratio="10" rot="SR0"/>
 </element>
+<element name="R6" library="rcl" package="R0603" value="100" x="14.25" y="32.25" rot="R180"/>
 </elements>
 <signals>
@@
 <signal name="LED_CMD">
 <contactref element="J1" pad="3"/>
-<contactref element="U1" pad="1"/>
-<wire x1="13.4398" y1="29.8422" x2="13.4398" y2="28.5602" width="0.3048" layer="1"/>
-<wire x1="13.4398" y1="28.5602" x2="13.75" y2="28.25" width="0.3048" layer="1"/>
-<via x="13.75" y="28.25" extent="1-16" drill="0.35"/>
-<wire x1="13.75" y1="28.25" x2="16.46" y2="25.54" width="0.3048" layer="16"/>
 <wire x1="16.46" y1="25.54" x2="19.75" y2="25.54" width="0.3048" layer="16"/>
+<contactref element="R6" pad="1"/>
+<wire x1="16.46" y1="25.54" x2="15" y2="27" width="0.3048" layer="16"/>
+<wire x1="15" y1="27" x2="15" y2="31" width="0.3048" layer="16"/>
+<via x="15" y="31" extent="1-16" drill="0.5"/>
+<wire x1="15" y1="31" x2="15" y2="32.15" width="0.3048" layer="1"/>
+<wire x1="15" y1="32.15" x2="15.1" y2="32.25" width="0.3048" layer="1"/>
 </signal>
 <signal name="LED_GND">
@@
 <wire x1="12.5" y1="27.6578" x2="12.5" y2="24.75" width="0.4064" layer="1"/>
 </signal>
+<signal name="N$6">
+<contactref element="R6" pad="2"/>
+<contactref element="U1" pad="1"/>
+<wire x1="13.4398" y1="29.8422" x2="13.4398" y2="32.2102" width="0.3048" layer="1"/>
+<wire x1="13.4398" y1="32.2102" x2="13.4" y2="32.25" width="0.3048" layer="1"/>
+</signal>
 </signals>
