File: VarmoEmergencyStop/Rev A1/VarmoEmergencyStop - Rev A1.brd (EAGLE design)
At the start: 95 x 25 mm, 6 parts, among them J1 22-05-7028-02, X1 NC3MAV, X2 NC3FAV2, X3 NC3MAV

Commit message: Generate Gerber
Parts:
- added J2: 22-05-7038-03, con-molex:7395-03
- moved J1 36.0 mm to (28.5, 5.50)
Connections:
- removed net GND-END: X1.1
- net +5V-THROUGH: now also J2.2
- net ES-END: now also J2.3
- net GND-THROUGH: now also J2.1, X1.1
Routing:
- net GND-THROUGH: track 43.7 -> 84.2 mm
- net +5V-THROUGH: track 34.0 -> 57.4 mm
- net ES-END: track 79.4 -> 85.1 mm
Changed lines of the file:
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@@
 <setting verticaltext="up"/>
 </settings>
-<grid distance="1" unitdist="mm" unit="mil" style="lines" multiple="1" display="no" altdistance="0.5" altunitdist="mm" altunit="mm"/>
+<grid distance="1" unitdist="mm" unit="mm" style="lines" multiple="1" display="no" altdistance="0.5" altunitdist="mm" altunit="mm"/>
 <layers>
 <layer number="1" name="Top" color="4" fill="1" visible="yes" active="yes"/>
@@
 <layer number="14" name="Route14" color="1" fill="6" visible="no" active="no"/>
 <layer number="15" name="Route15" color="4" fill="6" visible="no" active="no"/>
-<layer number="16" name="Bottom" color="1" fill="1" visible="yes" active="yes"/>
+<layer number="16" name="Bottom" color="1" fill="1" visible="no" active="yes"/>
 <layer number="17" name="Pads" color="2" fill="1" visible="yes" active="yes"/>
 <layer number="18" name="Vias" color="2" fill="1" visible="yes" active="yes"/>
@@
 <layer number="20" name="Dimension" color="15" fill="1" visible="yes" active="yes"/>
 <layer number="21" name="tPlace" color="7" fill="1" visible="yes" active="yes"/>
-<layer number="22" name="bPlace" color="7" fill="1" visible="yes" active="yes"/>
+<layer number="22" name="bPlace" color="7" fill="1" visible="no" active="yes"/>
 <layer number="23" name="tOrigins" color="15" fill="1" visible="yes" active="yes"/>
-<layer number="24" name="bOrigins" color="15" fill="1" visible="yes" active="yes"/>
+<layer number="24" name="bOrigins" color="15" fill="1" visible="no" active="yes"/>
 <layer number="25" name="tNames" color="7" fill="1" visible="yes" active="yes"/>
-<layer number="26" name="bNames" color="7" fill="1" visible="yes" active="yes"/>
-<layer number="27" name="tValues" color="7" fill="1" visible="no" active="yes"/>
+<layer number="26" name="bNames" color="7" fill="1" visible="no" active="yes"/>
+<layer number="27" name="tValues" color="7" fill="1" visible="yes" active="yes"/>
 <layer number="28" name="bValues" color="7" fill="1" visible="no" active="yes"/>
 <layer number="29" name="tStop" color="7" fill="3" visible="no" active="yes"/>
@@
 <layer number="49" name="Reference" color="7" fill="1" visible="yes" active="yes"/>
 <layer number="50" name="dxf" color="7" fill="1" visible="no" active="no"/>
-<layer number="51" name="tDocu" color="7" fill="1" visible="no" active="yes"/>
+<layer number="51" name="tDocu" color="7" fill="1" visible="yes" active="yes"/>
 <layer number="52" name="bDocu" color="7" fill="1" visible="no" active="yes"/>
 <layer number="53" name="tGND_GNDA" color="7" fill="1" visible="no" active="no"/>
@@
 </autorouter>
 <elements>
-<element name="J1" library="con-molex" package="7395-02" value="22-05-7028-02" x="64.5" y="5.5">
-<attribute name="OC_FARNELL" value="9731601" x="64.5" y="5.5" size="1.778" layer="27" display="off"/>
-<attribute name="OC_NEWARK" value="unknown" x="64.5" y="5.5" size="1.778" layer="27" display="off"/>
-<attribute name="MPN" value="" x="64.5" y="5.5" size="1.778" layer="27" display="off"/>
-<attribute name="MF" value="" x="64.5" y="5.5" size="1.778" layer="27" display="off"/>
+<element name="J1" library="con-molex" package="7395-02" value="22-05-7028-02" x="28.5" y="5.5">
+<attribute name="OC_FARNELL" value="9731601" x="28.5" y="5.5" size="1.778" layer="27" display="off"/>
+<attribute name="OC_NEWARK" value="unknown" x="28.5" y="5.5" size="1.778" layer="27" display="off"/>
+<attribute name="MPN" value="" x="28.5" y="5.5" size="1.778" layer="27" display="off"/>
+<attribute name="MF" value="" x="28.5" y="5.5" size="1.778" layer="27" display="off"/>
 </element>
 <element name="X1" library="con-neutrik_ag" package="NC3MAV" value="NC3MAV" x="84" y="12.5" smashed="yes">
@@
 <element name="U$1" library="exmachina" package="EXM-LOGO-BASELINE" value="EXMACHINA-LOGO-NAME" x="61" y="10" rot="R90"/>
 <element name="U$2" library="cc-by-sa" package="CC-BY-NC-SA" value="CC-BY-NC-SA" x="67" y="19" rot="R90"/>
+<element name="J2" library="con-molex" package="7395-03" value="22-05-7038-03" x="66" y="5">
+<attribute name="OC_NEWARK" value="unknown" x="66" y="5" size="1.778" layer="27" display="off"/>
+<attribute name="MPN" value="" x="66" y="5" size="1.778" layer="27" display="off"/>
+<attribute name="MF" value="" x="66" y="5" size="1.778" layer="27" display="off"/>
+<attribute name="OC_FARNELL" value="9731610 " x="66" y="5" size="1.778" layer="27" display="off"/>
+</element>
 </elements>
 <signals>
@@
 <contactref element="X3" pad="3"/>
 <wire x1="11" y1="8.05" x2="45" y2="8.05" width="0.8128" layer="1"/>
+<contactref element="J2" pad="2"/>
+<wire x1="45" y1="8.05" x2="64.95" y2="8.05" width="0.8128" layer="1"/>
+<wire x1="64.95" y1="8.05" x2="66" y2="7" width="0.8128" layer="1"/>
+<wire x1="66" y1="7" x2="66" y2="5" width="0.8128" layer="1"/>
 </signal>
 <signal name="GND" class="1">
@@
 </polygon>
 </signal>
-<signal name="GND-END" class="1">
-<contactref element="X1" pad="1"/>
-</signal>
 <signal name="ES-END" class="1">
 <contactref element="X1" pad="2"/>
@@
 <contactref element="X3" pad="2"/>
 <wire x1="14.81" y1="12.5" x2="17.31" y2="10" width="0.8128" layer="16"/>
-<wire x1="17.31" y1="10" x2="62" y2="10" width="0.8128" layer="16"/>
-<wire x1="62" y1="10" x2="63.23" y2="8.77" width="0.8128" layer="16"/>
-<wire x1="63.23" y1="8.77" x2="63.23" y2="5.5" width="0.8128" layer="16"/>
+<wire x1="17.31" y1="10" x2="28" y2="10" width="0.8128" layer="16"/>
+<wire x1="28" y1="10" x2="64" y2="10" width="0.8128" layer="16"/>
 <wire x1="87.81" y1="12.5" x2="85.31" y2="10" width="0.8128" layer="16"/>
-<wire x1="85.31" y1="10" x2="64.46" y2="10" width="0.8128" layer="16"/>
-<wire x1="64.46" y1="10" x2="63.23" y2="8.77" width="0.8128" layer="16"/>
+<wire x1="85.31" y1="10" x2="64" y2="10" width="0.8128" layer="16"/>
+<contactref element="J2" pad="3"/>
+<wire x1="63.46" y1="5" x2="63.46" y2="9.46" width="0.8128" layer="16"/>
+<wire x1="63.46" y1="9.46" x2="64" y2="10" width="0.8128" layer="16"/>
+<wire x1="27.23" y1="5.5" x2="27.23" y2="9.23" width="0.8128" layer="16"/>
+<wire x1="27.23" y1="9.23" x2="28" y2="10" width="0.8128" layer="16"/>
 </signal>
 <signal name="GND-THROUGH" class="1">
@@
 <wire x1="46.31" y1="15" x2="9.69" y2="15" width="0.8128" layer="1"/>
 <wire x1="9.69" y1="15" x2="7.19" y2="12.5" width="0.8128" layer="1"/>
+<contactref element="J2" pad="1"/>
+<wire x1="48.81" y1="12.5" x2="64" y2="12.5" width="0.8128" layer="1"/>
+<wire x1="64" y1="12.5" x2="64.5" y2="12.5" width="0.8128" layer="1"/>
+<wire x1="64.5" y1="12.5" x2="68.54" y2="8.46" width="0.8128" layer="1"/>
+<wire x1="68.54" y1="8.46" x2="68.54" y2="5" width="0.8128" layer="1"/>
+<contactref element="X1" pad="1"/>
+<wire x1="80.19" y1="12.5" x2="64.5" y2="12.5" width="0.8128" layer="1"/>
 </signal>
 </signals>
