File: Varmo/Rev A3/Varmo - Rev A3.brd (EAGLE design)
At the start: 127 x 90 mm, 108 parts, among them J1 22-05-7028-02, J2 22-05-7028-02, J3 22-05-7038-03, J4 22-05-7038-03, J5 22-05-7038-03, J6 22-05-7038-03, J7 22-05-7058-05, J9 22-05-7038-03, U1 90814-0210, U2 SN74LVC2G17DBVR, U3 SN74LVC2G17DBVR, U4 TPL0401A, U5 90814-0210, U8 M20DX256, X1 90814-0210, X2 90814-0210, X6 NC5MAV-SW, X7 90814-0210, X8 90814-0210

Commit message: Fix #8: Add filter and shmitt trigger to encoder inputs.
Parts:
- added C10, C17, C18, C19, C20, C21, C22, C23, C5, C6: 0.1uF, rcl:C0603
- added R37, R38, R39, R52, R55, R56, R57: 1k, rcl:R0603
- added U6: SN74LVC3G17DCTR, ti:SOP65P400X130-8N
- added U7, U9: SN74LVC2G17DBVR, ti:SOT95P280X145-6N
- moved U$6 46.3 mm to (73.2, 83.8)
- moved U$1 43.2 mm to (75.7, 75.8)
- moved C1 4.30 mm to (42.1, 28.8)
- moved L1 4.30 mm to (42.4, 25.2)
- moved U1 1.50 mm to (48.5, 27.5)
Connections:
- new net DIR_A_MCU: U7.6, U8.11
- new net DIR_B_MCU: U7.4, U8.10
- new net DIR_C_MCU: U8.9, U9.6
- new net DIR_D_MCU: U8.8, U9.4
- new net ENCODER_A_MCU: U6.1, U8.13
- new net ENCODER_B_MCU: U6.3, U8.14
- new net N$17: C10.1, R39.2, U7.1
- new net N$30: C17.1, R52.2, U7.3
- new net N$31: C5.1, R37.2, U9.1
- new net N$32: C6.1, R38.2, U9.3
- new net N$40: C20.1, R55.2, U6.7
- new net N$41: C21.1, R56.2, U6.5
- new net N$42: C22.1, R57.2, U6.2
- new net PUSH_MCU: U6.6, U8.12
- net +3V3: now also C18.1, C19.1, C23.1, U6.8, U7.5, U9.5
- net DIR_A: now also R39.1; no longer U8.11
- net DIR_B: now also R52.1; no longer U8.10
- net DIR_C: now also R37.1; no longer U8.9
- net DIR_D: now also R38.1; no longer U8.8
- net ENCODER_A: now also R55.1; no longer U8.13
- net ENCODER_B: now also R56.1; no longer U8.14
- net GND1: now also C10.2, C17.2, C18.2, C19.2, C20.2, C21.2, C22.2, C23.2, C5.2, C6.2, U6.4, U7.2, U9.2
- net PUSH: now also R57.1; no longer U8.12
Routing:
- net +3V3: track 0.00 -> 83.2 mm, vias 8 -> 10
- net PUSH_MCU: track 0.00 -> 38.9 mm, vias 0 -> 1
- net DIR_A: track 88.1 -> 56.1 mm, vias 2 -> 3
- net DIR_B: track 99.0 -> 69.1 mm, vias 4 -> 5
- net DIR_C: track 96.1 -> 68.0 mm, vias 2 -> 3
- net ENCODER_A_MCU: track 0.00 -> 28.0 mm, vias 0 -> 1
- net PUSH: track 88.9 -> 64.0 mm, vias 2 -> 1
- net ENCODER_B: track 101.2 -> 76.4 mm, vias 6 -> 7
- net ENCODER_B_MCU: track 0.00 -> 24.6 mm, vias 0 -> 1
- net DIR_D: track 97.2 -> 72.8 mm, vias 1 -> 3
- net DIR_D_MCU: track 0.00 -> 22.5 mm, vias 0 -> 1
- net DIR_B_MCU: track 0.00 -> 22.3 mm, vias 0 -> 1
- net DIR_C_MCU: track 0.00 -> 21.6 mm, vias 0 -> 1
- net DIR_A_MCU: track 0.00 -> 21.2 mm, vias 0 -> 1
- net ENCODER_A: track 97.5 -> 77.5 mm, vias 3 -> 5
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Other:
- board size 127 x 90 mm -> 126 x 90 mm
