File: WDY/Main_Board/Rev A1/Main_Board.sch (EAGLE design)
At the start: 174 parts, among them J1 22-05-7028-02, J10 22-05-7038-03, J11 22-05-7028-02, J12 22-05-7028-02, J13 22-05-7028-02, J14 22-05-7028-02, J15 22-05-7058-05, J2 22-05-7028-02, J3 22-05-7048-04, J4 22-05-7048-04, J5 1241050-5, J6 90814-0208, J7 90814-0206, J8 90814-0208, J9 22-05-7038-03, K1 G6K-2G-Y, K2 G6K-2G-Y, K3 G6K-2G-Y, K4 G6K-2G-Y, P1 RB1-125BAG1A, U1 LPC1768FBD100, U11 SN74LVC3G17DCTR, U2 SN74LVC3G17DCTR, U3 SN74LVC3G17DCTR, U4 TPL0401A, U5 AT24C512C-SSHM-B, U6 SN74LVC2G17DBVR, U7 SN74LVC2G17DBVR, U8 LT1767EMS8E-5PBF, U9 TC1264-3.3, X1 FC-135, X2 MSTBA2

Commit message: Main_Board : Add the revision on the folder
Connections:
- removed net CAN_V+: U$5C.9
- removed net N$1: C1.1, R3.1, R4.1
- removed net N$2: C2.1, R5.1, R6.1
- net +24V: now also U$5C.9
- net +3V3: now also C1.1, C2.1, R3.1, R4.1, R5.1, R6.1
- net EEPROM_SCL: no longer U1.P0[11]/RXD2/SCL2/MAT3[1]
- net EEPROM_SDA: no longer U1.P0[10]/TXD2/SDA2/MAT3[0]
- net HMI_BUTTON_1: no longer U1.P0[16]/RXD1/SSEL0/SSEL
- net HMI_BUTTON_2: no longer U1.P0[15]/TXD1/SCK0/SCK
- net HMI_BUTTON_3: no longer U1.P0[17]/CTS1/MISO0/MISO
- net HMI_BUTTON_4: no longer U1.P0[18]/DCD1/MOSI0/MOSI
- net HMI_BUTTON_5: no longer U1.P0[19]/DSR1/SDA1
- net HMI_BUTTON_6: no longer U1.P0[20]/DTR1/SCL1
- net HMI_BUTTON_CPU_1: now also U1.P0[16]/RXD1/SSEL0/SSEL
- net HMI_BUTTON_CPU_2: now also U1.P0[15]/TXD1/SCK0/SCK
- net HMI_BUTTON_CPU_3: now also U1.P0[17]/CTS1/MISO0/MISO
- net HMI_BUTTON_CPU_4: now also U1.P0[18]/DCD1/MOSI0/MOSI
- net HMI_BUTTON_CPU_5: now also U1.P0[19]/DSR1/SDA1
- net HMI_BUTTON_CPU_6: now also U1.P0[20]/DTR1/SCL1
- net HMI_LCD_SCL: now also U1.P0[11]/RXD2/SCL2/MAT3[1]; no longer U1.P0[28]/SCL0/USB_SCL
- net HMI_LCD_SDA: now also U1.P0[10]/TXD2/SDA2/MAT3[0]; no longer U1.P0[27]/SDA0/USB_SDA
Changed lines of the file:
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@@
 <part name="R61" library="rcl" deviceset="R-EU_" device="R0603" value="4k7"/>
 <part name="C54" library="rcl" deviceset="C-EU" device="C0603" value="0.1uF"/>
+<part name="P+21" library="supply3" deviceset="+24V" device=""/>
 </parts>
 <sheets>
@@
 <instance part="P+15" gate="1" x="35.56" y="147.32"/>
 <instance part="GND62" gate="1" x="35.56" y="129.54"/>
+<instance part="P+21" gate="1" x="96.52" y="83.82"/>
 </instances>
 <busses>
 </busses>
 <nets>
-<net name="N$1" class="0">
-<segment>
-<pinref part="C1" gate="G$1" pin="1"/>
-<pinref part="R3" gate="G$1" pin="1"/>
-<wire x1="106.68" y1="170.18" x2="106.68" y2="177.8" width="0.1524" layer="91"/>
-<pinref part="R4" gate="G$1" pin="1"/>
-<wire x1="106.68" y1="177.8" x2="114.3" y2="177.8" width="0.1524" layer="91"/>
-<junction x="106.68" y="177.8"/>
-</segment>
-</net>
-<net name="N$2" class="0">
-<segment>
-<pinref part="C2" gate="G$1" pin="1"/>
-<pinref part="R5" gate="G$1" pin="1"/>
-<wire x1="124.46" y1="170.18" x2="124.46" y2="177.8" width="0.1524" layer="91"/>
-<pinref part="R6" gate="G$1" pin="1"/>
-<wire x1="124.46" y1="177.8" x2="132.08" y2="177.8" width="0.1524" layer="91"/>
-<junction x="124.46" y="177.8"/>
-</segment>
-</net>
 <net name="ETH_TX_P" class="1">
 <segment>
@@
 <wire x1="71.12" y1="175.26" x2="78.74" y2="175.26" width="0.1524" layer="91"/>
 <junction x="78.74" y="175.26"/>
+<pinref part="C1" gate="G$1" pin="1"/>
+<pinref part="R3" gate="G$1" pin="1"/>
+<wire x1="106.68" y1="170.18" x2="106.68" y2="175.26" width="0.1524" layer="91"/>
+<pinref part="R4" gate="G$1" pin="1"/>
+<wire x1="106.68" y1="175.26" x2="106.68" y2="177.8" width="0.1524" layer="91"/>
+<wire x1="106.68" y1="177.8" x2="114.3" y2="177.8" width="0.1524" layer="91"/>
+<junction x="106.68" y="177.8"/>
+<wire x1="78.74" y1="175.26" x2="106.68" y2="175.26" width="0.1524" layer="91"/>
+<junction x="106.68" y="175.26"/>
+<pinref part="C2" gate="G$1" pin="1"/>
+<pinref part="R5" gate="G$1" pin="1"/>
+<wire x1="124.46" y1="170.18" x2="124.46" y2="175.26" width="0.1524" layer="91"/>
+<pinref part="R6" gate="G$1" pin="1"/>
+<wire x1="124.46" y1="175.26" x2="124.46" y2="177.8" width="0.1524" layer="91"/>
+<wire x1="124.46" y1="177.8" x2="132.08" y2="177.8" width="0.1524" layer="91"/>
+<junction x="124.46" y="177.8"/>
+<wire x1="106.68" y1="175.26" x2="124.46" y2="175.26" width="0.1524" layer="91"/>
+<junction x="124.46" y="175.26"/>
 </segment>
 <segment>
@@
 </segment>
 </net>
-<net name="CAN_V+" class="0">
-<segment>
-<pinref part="U$5" gate="C" pin="9"/>
-<wire x1="91.44" y1="66.04" x2="99.06" y2="66.04" width="0.1524" layer="91"/>
-<label x="99.06" y="66.04" size="1.27" layer="95" xref="yes"/>
-</segment>
-</net>
 <net name="N$6" class="0">
 <segment>
@@
 <wire x1="27.94" y1="139.7" x2="35.56" y2="139.7" width="0.1524" layer="91"/>
 <wire x1="35.56" y1="139.7" x2="35.56" y2="144.78" width="0.1524" layer="91"/>
+</segment>
+</net>
+<net name="+24V" class="0">
+<segment>
+<pinref part="U$5" gate="C" pin="9"/>
+<pinref part="P+21" gate="1" pin="+24V"/>
+<wire x1="91.44" y1="66.04" x2="96.52" y2="66.04" width="0.1524" layer="91"/>
+<wire x1="96.52" y1="66.04" x2="96.52" y2="81.28" width="0.1524" layer="91"/>
 </segment>
 </net>
@@
 </segment>
 <segment>
-<pinref part="U1" gate="A" pin="P0[10]/TXD2/SDA2/MAT3[0]"/>
-<wire x1="132.08" y1="114.3" x2="124.46" y2="114.3" width="0.1524" layer="91"/>
-<label x="124.46" y="114.3" size="1.27" layer="95" rot="R180" xref="yes"/>
+<wire x1="132.08" y1="172.72" x2="124.46" y2="172.72" width="0.1524" layer="91"/>
+<label x="124.46" y="172.72" size="1.27" layer="95" rot="R180" xref="yes"/>
 </segment>
 </net>
@@
 </segment>
 <segment>
+<wire x1="132.08" y1="175.26" x2="124.46" y2="175.26" width="0.1524" layer="91"/>
+<label x="124.46" y="175.26" size="1.27" layer="95" rot="R180" xref="yes"/>
+</segment>
+</net>
+<net name="HMI_LCD_SCL" class="1">
+<segment>
+<label x="124.46" y="111.76" size="1.27" layer="95" rot="R180" xref="yes"/>
 <pinref part="U1" gate="A" pin="P0[11]/RXD2/SCL2/MAT3[1]"/>
 <wire x1="132.08" y1="111.76" x2="124.46" y2="111.76" width="0.1524" layer="91"/>
-<label x="124.46" y="111.76" size="1.27" layer="95" rot="R180" xref="yes"/>
-</segment>
-</net>
-<net name="HMI_LCD_SCL" class="1">
-<segment>
-<pinref part="U1" gate="A" pin="P0[28]/SCL0/USB_SCL"/>
-<wire x1="132.08" y1="175.26" x2="124.46" y2="175.26" width="0.1524" layer="91"/>
-<label x="124.46" y="175.26" size="1.27" layer="95" rot="R180" xref="yes"/>
 </segment>
 </net>
 <net name="HMI_LCD_SDA" class="1">
 <segment>
-<pinref part="U1" gate="A" pin="P0[27]/SDA0/USB_SDA"/>
-<wire x1="132.08" y1="172.72" x2="124.46" y2="172.72" width="0.1524" layer="91"/>
-<label x="124.46" y="172.72" size="1.27" layer="95" rot="R180" xref="yes"/>
-</segment>
-</net>
-<net name="HMI_BUTTON_2" class="1">
-<segment>
-<pinref part="U1" gate="A" pin="P0[15]/TXD1/SCK0/SCK"/>
-<wire x1="314.96" y1="137.16" x2="320.04" y2="137.16" width="0.1524" layer="91"/>
-<label x="320.04" y="137.16" size="1.27" layer="95" xref="yes"/>
-</segment>
-</net>
-<net name="HMI_BUTTON_3" class="1">
-<segment>
-<pinref part="U1" gate="A" pin="P0[17]/CTS1/MISO0/MISO"/>
-<wire x1="314.96" y1="134.62" x2="320.04" y2="134.62" width="0.1524" layer="91"/>
-<label x="320.04" y="134.62" size="1.27" layer="95" xref="yes"/>
-</segment>
-</net>
-<net name="HMI_BUTTON_4" class="1">
-<segment>
-<pinref part="U1" gate="A" pin="P0[18]/DCD1/MOSI0/MOSI"/>
-<wire x1="314.96" y1="132.08" x2="320.04" y2="132.08" width="0.1524" layer="91"/>
-<label x="320.04" y="132.08" size="1.27" layer="95" xref="yes"/>
-</segment>
-</net>
-<net name="HMI_BUTTON_1" class="1">
-<segment>
-<pinref part="U1" gate="A" pin="P0[16]/RXD1/SSEL0/SSEL"/>
-<wire x1="314.96" y1="139.7" x2="320.04" y2="139.7" width="0.1524" layer="91"/>
-<label x="320.04" y="139.7" size="1.27" layer="95" xref="yes"/>
-</segment>
-</net>
-<net name="HMI_BUTTON_5" class="1">
-<segment>
-<pinref part="U1" gate="A" pin="P0[19]/DSR1/SDA1"/>
-<wire x1="314.96" y1="129.54" x2="320.04" y2="129.54" width="0.1524" layer="91"/>
-<label x="320.04" y="129.54" size="1.27" layer="95" xref="yes"/>
-</segment>
-</net>
-<net name="HMI_BUTTON_6" class="0">
-<segment>
-<pinref part="U1" gate="A" pin="P0[20]/DTR1/SCL1"/>
-<wire x1="314.96" y1="127" x2="320.04" y2="127" width="0.1524" layer="91"/>
-<label x="320.04" y="127" size="1.27" layer="95" xref="yes"/>
+<label x="124.46" y="114.3" size="1.27" layer="95" rot="R180" xref="yes"/>
+<pinref part="U1" gate="A" pin="P0[10]/TXD2/SDA2/MAT3[0]"/>
+<wire x1="124.46" y1="114.3" x2="132.08" y2="114.3" width="0.1524" layer="91"/>
 </segment>
 </net>
@@
 </segment>
 </net>
+<net name="HMI_BUTTON_CPU_1" class="0">
+<segment>
+<pinref part="U1" gate="A" pin="P0[16]/RXD1/SSEL0/SSEL"/>
+<wire x1="314.96" y1="139.7" x2="320.04" y2="139.7" width="0.1524" layer="91"/>
+<label x="320.04" y="139.7" size="1.27" layer="95" xref="yes"/>
+</segment>
+</net>
+<net name="HMI_BUTTON_CPU_2" class="0">
+<segment>
+<pinref part="U1" gate="A" pin="P0[15]/TXD1/SCK0/SCK"/>
+<wire x1="314.96" y1="137.16" x2="320.04" y2="137.16" width="0.1524" layer="91"/>
+<label x="320.04" y="137.16" size="1.27" layer="95" xref="yes"/>
+</segment>
+</net>
+<net name="HMI_BUTTON_CPU_3" class="0">
+<segment>
+<pinref part="U1" gate="A" pin="P0[17]/CTS1/MISO0/MISO"/>
+<wire x1="314.96" y1="134.62" x2="320.04" y2="134.62" width="0.1524" layer="91"/>
+<label x="320.04" y="134.62" size="1.27" layer="95" xref="yes"/>
+</segment>
+</net>
+<net name="HMI_BUTTON_CPU_4" class="0">
+<segment>
+<pinref part="U1" gate="A" pin="P0[18]/DCD1/MOSI0/MOSI"/>
+<wire x1="314.96" y1="132.08" x2="320.04" y2="132.08" width="0.1524" layer="91"/>
+<label x="320.04" y="132.08" size="1.27" layer="95" xref="yes"/>
+</segment>
+</net>
+<net name="HMI_BUTTON_CPU_5" class="0">
+<segment>
+<pinref part="U1" gate="A" pin="P0[19]/DSR1/SDA1"/>
+<wire x1="314.96" y1="129.54" x2="320.04" y2="129.54" width="0.1524" layer="91"/>
+<label x="320.04" y="129.54" size="1.27" layer="95" xref="yes"/>
+</segment>
+</net>
+<net name="HMI_BUTTON_CPU_6" class="0">
+<segment>
+<pinref part="U1" gate="A" pin="P0[20]/DTR1/SCL1"/>
+<wire x1="314.96" y1="127" x2="320.04" y2="127" width="0.1524" layer="91"/>
+<label x="320.04" y="127" size="1.27" layer="95" xref="yes"/>
+</segment>
+</net>

Commit message: Route the signal of USB, CAN, ETH, Relay, LED, Button, ADC
Parts:
- added R62, R63, R64, R65: 100, rcl:R-EU_R0603
- C32: value 18pF -> 0.1uF
Connections:
- removed net GND1: LED5.C
- new net N$1: J7.3, R64.1
- new net N$2: J7.5, R65.1
- new net N$63: J7.2, R62.2
- new net N$64: J7.4, R63.2
- net GND: now also LED5.C
- net HMI_LED_1: now also R62.1; no longer J7.2
- net HMI_LED_2: now also R64.2; no longer J7.3
- net HMI_LED_3: now also R63.1; no longer J7.4
- net HMI_LED_4: now also R65.2; no longer J7.5
Changed lines of the file:
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@@
 <part name="C31" library="rcl" deviceset="C-EU" device="C0603" value="18pF"/>
 <part name="L1" library="coilcraft" deviceset="0603PS" device="" value="0603PS-103KLB"/>
-<part name="C32" library="rcl" deviceset="C-EU" device="C0603" value="18pF"/>
+<part name="C32" library="rcl" deviceset="C-EU" device="C0603" value="0.1uF"/>
 <part name="+3V19" library="supply1" deviceset="+3V3" device=""/>
 <part name="GND59" library="supply1" deviceset="GND" device=""/>
@@
 <part name="C54" library="rcl" deviceset="C-EU" device="C0603" value="0.1uF"/>
 <part name="P+21" library="supply3" deviceset="+24V" device=""/>
+<part name="R62" library="rcl" deviceset="R-EU_" device="R0603" value="100"/>
+<part name="R63" library="rcl" deviceset="R-EU_" device="R0603" value="100"/>
+<part name="R64" library="rcl" deviceset="R-EU_" device="R0603" value="100"/>
+<part name="R65" library="rcl" deviceset="R-EU_" device="R0603" value="100"/>
 </parts>
 <sheets>
@@
 <instance part="GND77" gate="1" x="144.78" y="231.14"/>
 <instance part="P+22" gate="1" x="144.78" y="254"/>
+<instance part="R62" gate="G$1" x="325.12" y="228.6" smashed="yes" rot="R180">
+<attribute name="NAME" x="321.31" y="230.6574" size="1.778" layer="95" rot="R180"/>
+<attribute name="VALUE" x="334.01" y="230.632" size="1.778" layer="96" rot="R180"/>
+</instance>
+<instance part="R63" gate="G$1" x="325.12" y="226.06" smashed="yes" rot="R180">
+<attribute name="NAME" x="321.31" y="228.1174" size="1.778" layer="95" rot="R180"/>
+<attribute name="VALUE" x="334.01" y="228.092" size="1.778" layer="96" rot="R180"/>
+</instance>
+<instance part="R64" gate="G$1" x="266.7" y="226.06" smashed="yes" rot="R180">
+<attribute name="NAME" x="262.89" y="228.1174" size="1.778" layer="95" rot="R180"/>
+<attribute name="VALUE" x="275.59" y="228.092" size="1.778" layer="96" rot="R180"/>
+</instance>
+<instance part="R65" gate="G$1" x="266.7" y="223.52" smashed="yes" rot="R180">
+<attribute name="NAME" x="262.89" y="225.5774" size="1.778" layer="95" rot="R180"/>
+<attribute name="VALUE" x="275.59" y="225.552" size="1.778" layer="96" rot="R180"/>
+</instance>
 </instances>
 <busses>
@@
 <net name="HMI_LED_1" class="1">
 <segment>
-<pinref part="J7" gate="A" pin="2"/>
-<wire x1="314.96" y1="228.6" x2="322.58" y2="228.6" width="0.1524" layer="91"/>
-<label x="322.58" y="228.6" size="1.27" layer="95" xref="yes"/>
+<label x="340.36" y="228.6" size="1.27" layer="95" xref="yes"/>
+<pinref part="R62" gate="G$1" pin="1"/>
+<wire x1="330.2" y1="228.6" x2="340.36" y2="228.6" width="0.1524" layer="91"/>
 </segment>
 </net>
 <net name="HMI_LED_2" class="1">
 <segment>
-<pinref part="J7" gate="A" pin="3"/>
-<wire x1="279.4" y1="226.06" x2="271.78" y2="226.06" width="0.1524" layer="91"/>
-<label x="271.78" y="226.06" size="1.27" layer="95" rot="R180" xref="yes"/>
+<label x="256.54" y="226.06" size="1.27" layer="95" rot="R180" xref="yes"/>
+<pinref part="R64" gate="G$1" pin="2"/>
+<wire x1="261.62" y1="226.06" x2="256.54" y2="226.06" width="0.1524" layer="91"/>
 </segment>
 </net>
 <net name="HMI_LED_3" class="1">
 <segment>
-<pinref part="J7" gate="A" pin="4"/>
-<wire x1="314.96" y1="226.06" x2="322.58" y2="226.06" width="0.1524" layer="91"/>
-<label x="322.58" y="226.06" size="1.27" layer="95" xref="yes"/>
+<label x="340.36" y="226.06" size="1.27" layer="95" xref="yes"/>
+<pinref part="R63" gate="G$1" pin="1"/>
+<wire x1="330.2" y1="226.06" x2="340.36" y2="226.06" width="0.1524" layer="91"/>
 </segment>
 </net>
 <net name="HMI_LED_4" class="1">
 <segment>
-<pinref part="J7" gate="A" pin="5"/>
-<wire x1="279.4" y1="223.52" x2="271.78" y2="223.52" width="0.1524" layer="91"/>
-<label x="271.78" y="223.52" size="1.27" layer="95" rot="R180" xref="yes"/>
+<label x="256.54" y="223.52" size="1.27" layer="95" rot="R180" xref="yes"/>
+<pinref part="R65" gate="G$1" pin="2"/>
+<wire x1="261.62" y1="223.52" x2="256.54" y2="223.52" width="0.1524" layer="91"/>
 </segment>
 </net>
@@
 </segment>
 </net>
+<net name="N$1" class="0">
+<segment>
+<pinref part="R64" gate="G$1" pin="1"/>
+<pinref part="J7" gate="A" pin="3"/>
+<wire x1="271.78" y1="226.06" x2="279.4" y2="226.06" width="0.1524" layer="91"/>
+</segment>
+</net>
+<net name="N$2" class="0">
+<segment>
+<pinref part="R65" gate="G$1" pin="1"/>
+<pinref part="J7" gate="A" pin="5"/>
+<wire x1="271.78" y1="223.52" x2="279.4" y2="223.52" width="0.1524" layer="91"/>
+</segment>
+</net>
+<net name="N$63" class="0">
+<segment>
+<pinref part="J7" gate="A" pin="2"/>
+<pinref part="R62" gate="G$1" pin="2"/>
+<wire x1="314.96" y1="228.6" x2="320.04" y2="228.6" width="0.1524" layer="91"/>
+</segment>
+</net>
+<net name="N$64" class="0">
+<segment>
+<pinref part="J7" gate="A" pin="4"/>
+<pinref part="R63" gate="G$1" pin="2"/>
+<wire x1="314.96" y1="226.06" x2="320.04" y2="226.06" width="0.1524" layer="91"/>
+</segment>
+</net>
 </nets>
 </sheet>
@@
 <segment>
 <pinref part="C43" gate="G$1" pin="-"/>
-<wire x1="127" y1="144.78" x2="127" y2="139.7" width="0.1524" layer="91"/>
+<wire x1="127" y1="144.78" x2="127" y2="142.24" width="0.1524" layer="91"/>
 <pinref part="GND67" gate="1" pin="GND"/>
+<pinref part="LED5" gate="G$1" pin="C"/>
+<wire x1="127" y1="142.24" x2="127" y2="139.7" width="0.1524" layer="91"/>
+<wire x1="147.32" y1="142.24" x2="147.32" y2="144.78" width="0.1524" layer="91"/>
+<wire x1="147.32" y1="142.24" x2="127" y2="142.24" width="0.1524" layer="91"/>
+<junction x="127" y="142.24"/>
 </segment>
 <segment>
@@
 </segment>
 </net>
-<net name="GND1" class="2">
-<segment>
-<pinref part="LED5" gate="G$1" pin="C"/>
-<wire x1="147.32" y1="142.24" x2="147.32" y2="144.78" width="0.1524" layer="91"/>
-<wire x1="147.32" y1="142.24" x2="127" y2="142.24" width="0.1524" layer="91"/>
-</segment>
-</net>

Commit message: #RW1 Schematics :  Ethernet clock 12MHz -> 50MHz  ETH_CLK_EN: useless signal  Forgotten connection to +3V3 of ethernet filters (@1.B3)  Pullup on AT24 WP and Test pads intead of solder jumper (@2.E1)  Missing Xtal @2.B3 (ASE-12)  Wrong connection between ETH_X1 and XTAL1 (@2.A1)  VREFN must be connected to ground  Switch between R12-R14 and Thermistors  Set R12-R14 to 10k  Add RTC backup battery  Add onboard reset button  Add onboard boot button  Add current limiting for LEDs outputs  Missing ground connection on LED5  Add transistor to switch off the LCB backlight
Parts:
- removed C31: 18pF, rcl:C-EUC0603
- added C55: 0.1uF, rcl:C-EUC0603
- added R66: 4k7, rcl:R-EU_R0603
- added R67: 10K, rcl:R-EU_R0603
- added R68, R69: 0R, rcl:R-EU_R0603
- added R70: 100, rcl:R-EU_R0603
- added SW1, SW2: B3FS-1015, Switch_SMT:B3FS-1015
- added T1: MMBT2222AL, transistor:MMBT2222AL
- added U$10: ASE-12, crystal:ASE
- added U$14: 3000, keystone:3000
- R11: value 10k -> 10K
- R12, R14, R43: value 4k7 -> 10k
- R28: value 50 -> 33
- SJ3: value (none) -> SOLDERJUMPERNC2; device jumper:SJ2W -> SparkFun-Passives:SOLDERJUMPERNC2
- U$3: value ASE_12 -> ASE_50
Connections:
- removed net CAN_STBY: R11.2
- removed net ISP_SELECT: U1.P2[10]/*EINT0/NMI
- removed net N$10: J1-1.S, R12.1, R13.2
- removed net N$31: J11-1.S, R43.2, R44.1
- removed net RESET\: U1.*RESET
- new net BOOT_SELECT: R67.1, SW2.1, U1.P2[10]/*EINT0/NMI
- new net HMI_LCD_BACKLIGHT: R70.2
- new net N$65: J1-2.S, R12.2
- new net N$66: J2-2.S, R14.1
- new net N$67: J11-2.S, R43.1
- new net RESET: R11.1, R68.1, SW1.1, U1.*RESET
- new net VBAT+: U$14.VBAT+
- net +3V3: now also C55.1, R11.2, R66.2, R67.2, U$10.VDD, U1.VREFN; no longer R12.2, R14.1, R43.1, SJ3.3
- net AVDD: now also J1-1.S, J11-1.S, J2-1.S, R13.2, R15.1, R44.1
- net ENCODER_A: now also U1.P1[20]/MCI0/PWM1[2]/SCK0; no longer U1.P2[6]/PCAP1[0]/RI1/TRACECLK
- net ENCODER_B: now also U1.P1[23]/MCI1/PWM1[4]/MISO0; no longer U1.P2[7]/RD2/RTS1
- net ENCODER_Z: now also U1.P1[24]/MCI2/PWM1[5]/MOSI0; no longer U1.P2[8]/TD2/TXD2
- net ETH_CLK_EN: no longer U$3.TRI
- net ETH_X1: no longer C31.1
- net GND: now also C55.2, R12.1, R14.2, R43.2, SW1.2, SW2.2, T1.E, U$10.GND, U$10.TRI, U$14.VBAT-, U$3.TRI, U$4.STBY; no longer J1-2.S, J11-2.S, J2-2.S
- net HMI_BUTTON_CPU_6: now also R68.2, R69.1; no longer U1.P0[20]/DTR1/SCL1
- net HMI_LCD_LED+: now also T1.C
- net N$22: now also R66.1
- net N$5: now also R69.2, U1.P0[20]/DTR1/SCL1; no longer R11.1, U$4.STBY
- net N$7: now also R70.1, T1.B; no longer J2-1.S, R14.2, R15.1
- net XTAL1: now also U$10.OUT; no longer C31.2
Other:
- moved on the sheet: C15, C16, C17, C18, C19, C20, C21, C22, C29, C30, C32, C33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
