File: ArmazConnect/Rev B4/ArmazConnect - Rev B4.brd (EAGLE design)
At the start: 160 x 31.5 mm, 54 parts, among them J1 22-05-7028-02, X0 NC3FAV2, X1 NC3FAV2, X2 NC3FAV2, X3 NC3FAV2, X4 NC5FAV-SW, X5 90814-0210, X8 87832-26

Commit message: Generate Gerber
Parts:
- removed U$2: CC-BY-SA, cc-by-sa:CC-BY-SA
- added CC1: CC-BY-NC-SA, cc-by-sa:CC-BY-NC-SA
Other:
- board text removed: "ArmazConnect Rev B3"
- board text removed: "Ethernet module power"
Changed lines of the file:
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@@
 <layer number="14" name="Route14" color="1" fill="6" visible="no" active="no"/>
 <layer number="15" name="Route15" color="19" fill="6" visible="no" active="no"/>
-<layer number="16" name="Bottom" color="21" fill="1" visible="yes" active="yes"/>
+<layer number="16" name="Bottom" color="21" fill="1" visible="no" active="yes"/>
 <layer number="17" name="Pads" color="18" fill="1" visible="yes" active="yes"/>
 <layer number="18" name="Vias" color="38" fill="1" visible="yes" active="yes"/>
@@
 <layer number="20" name="Dimension" color="7" fill="1" visible="yes" active="yes"/>
 <layer number="21" name="tPlace" color="55" fill="1" visible="yes" active="yes"/>
-<layer number="22" name="bPlace" color="54" fill="1" visible="yes" active="yes"/>
+<layer number="22" name="bPlace" color="54" fill="1" visible="no" active="yes"/>
 <layer number="23" name="tOrigins" color="15" fill="1" visible="yes" active="yes"/>
-<layer number="24" name="bOrigins" color="15" fill="1" visible="yes" active="yes"/>
-<layer number="25" name="tNames" color="55" fill="1" visible="no" active="yes"/>
+<layer number="24" name="bOrigins" color="15" fill="1" visible="no" active="yes"/>
+<layer number="25" name="tNames" color="55" fill="1" visible="yes" active="yes"/>
 <layer number="26" name="bNames" color="54" fill="1" visible="no" active="yes"/>
-<layer number="27" name="tValues" color="53" fill="1" visible="no" active="yes"/>
+<layer number="27" name="tValues" color="53" fill="1" visible="yes" active="yes"/>
 <layer number="28" name="bValues" color="52" fill="1" visible="no" active="yes"/>
 <layer number="29" name="tStop" color="7" fill="3" visible="no" active="yes"/>
@@
 <layer number="49" name="Reference" color="48" fill="1" visible="yes" active="yes"/>
 <layer number="50" name="dxf" color="7" fill="1" visible="no" active="no"/>
-<layer number="51" name="tDocu" color="55" fill="1" visible="no" active="yes"/>
+<layer number="51" name="tDocu" color="55" fill="1" visible="yes" active="yes"/>
 <layer number="52" name="bDocu" color="54" fill="1" visible="no" active="yes"/>
 <layer number="53" name="tGND_GNDA" color="7" fill="1" visible="no" active="no"/>
@@
 <wire x1="46" y1="58.27" x2="46" y2="19.27" width="0" layer="47"/>
 <wire x1="80" y1="58.27" x2="80" y2="19.27" width="0" layer="47"/>
-<text x="45.974" y="32.004" size="1.27" layer="25" ratio="10" align="bottom-center">DMX In</text>
-<text x="80.264" y="33.02" size="1.27" layer="25" ratio="10" align="bottom-center">DMX Out</text>
+<text x="28.746" y="22.224" size="1.27" layer="25" ratio="10" rot="R90" align="bottom-center">DMX In</text>
+<text x="62.98" y="22.014" size="1.27" layer="25" ratio="10" rot="R90" align="bottom-center">DMX Out</text>
 <text x="12.446" y="42.418" size="1.27" layer="25" ratio="10" align="bottom-center">Drive En</text>
 <text x="45.974" y="42.418" size="1.27" layer="25" ratio="10" align="bottom-center">Ext SW1</text>
@@
 <text x="114.3" y="42.418" size="1.27" layer="25" ratio="10" align="bottom-center">Ext SW3</text>
 <text x="148.082" y="42.418" size="1.27" layer="25" ratio="10" align="bottom-center">Remote link</text>
-<text x="106.68" y="66.548" size="1.27" layer="26" ratio="10" rot="MR0" align="bottom-center">Ethernet module power</text>
-<text x="61.976" y="61.214" size="1.016" layer="26" rot="MR0" align="top-left">ArmazConnect
-Rev B3</text>
 <text x="84.25" y="21.25" size="1.016" layer="22" font="vector" ratio="10" rot="MR0" align="top-left">ArmazConnect
 Rev B4</text>
@@
 <attribute name="MPN" value="" x="84" y="21" size="1.778" layer="28" rot="MR0" display="off"/>
 </element>
-<element name="U$2" library="cc-by-sa" package="CC-BY-SA" value="CC-BY-SA" x="93" y="21" rot="MR0">
-<attribute name="OC_FARNELL" value="unknown" x="93" y="21" size="1.778" layer="28" rot="MR0" display="off"/>
-<attribute name="MF" value="" x="93" y="21" size="1.778" layer="28" rot="MR0" display="off"/>
-<attribute name="MPN" value="" x="93" y="21" size="1.778" layer="28" rot="MR0" display="off"/>
-</element>
 <element name="R5" library="rcl" package="R0603" value="4K7, DNI" x="117.75" y="26" rot="R270">
 <attribute name="MPN" value="MCMR04X3301FTL" x="117.75" y="26" size="0.2032" layer="27" rot="R270" display="off"/>
@@
 <attribute name="OC_FARNELL" value="1716770" x="17" y="34.875" size="1.016" layer="27" rot="R270" display="off"/>
 </element>
+<element name="CC1" library="cc-by-sa" package="CC-BY-NC-SA" value="CC-BY-NC-SA" x="98.25" y="19.5" rot="MR0"/>
 </elements>
 <signals>
