File: ArmazConnect/Rev B4/ArmazConnect - Rev B4.sch (EAGLE design)
At the start: 54 parts, among them J1 22-05-7028-02, X0 NC3FAV2, X1 NC3FAV2, X2 NC3FAV2, X3 NC3FAV2, X4 NC5FAV-SW, X5 90814-0210, X8 87832-26

Commit message: Generate Gerber
Parts:
- removed U$2: CC-BY-SA, cc-by-sa:CC-BY-SA
- added CC1: CC-BY-NC-SA, cc-by-sa:CC-BY-NC-SA
Changed lines of the file:
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@@
-<attribute name="OC_FARNELL" value="unknown"/>
-</part>
-<part name="U$2" library="cc-by-sa" deviceset="CC-BY-SA" device="">
-<attribute name="MF" value=""/>
-<attribute name="MPN" value=""/>
 <attribute name="OC_FARNELL" value="unknown"/>
 </part>
@@
 <part name="+3V6" library="supply3" deviceset="VDD33A1" device=""/>
 <part name="SUPPLY13" library="supply2" deviceset="GND1" device=""/>
+<part name="CC1" library="cc-by-sa" deviceset="CC-BY-NC-SA" device=""/>
 </parts>
 <sheets>
@@
 <attribute name="MPN" x="358.14" y="30.48" size="1.778" layer="96" display="off"/>
 </instance>
-<instance part="U$2" gate="A" x="269.24" y="10.16">
-<attribute name="OC_FARNELL" x="269.24" y="10.16" size="1.778" layer="96" display="off"/>
-<attribute name="MF" x="269.24" y="10.16" size="1.778" layer="96" display="off"/>
-<attribute name="MPN" x="269.24" y="10.16" size="1.778" layer="96" display="off"/>
-</instance>
 <instance part="+3V4" gate="G$1" x="167.64" y="200.66"/>
 <instance part="SUPPLY6" gate="G$1" x="167.64" y="165.1"/>
@@
 <instance part="+3V6" gate="G$1" x="213.36" y="40.64" rot="R180"/>
 <instance part="SUPPLY13" gate="G$1" x="325.12" y="121.92"/>
+<instance part="CC1" gate="G$1" x="302.26" y="10.16"/>
 </instances>
 <busses>
