File: ArmazCape/Rev B4/ArmazCape - Rev B4.sch (EAGLE design)
At the start: 167 parts, among them IC1 AT93C46EN-SH-BSOIC8, P1 RB1-125BAG1A, Q1 32.768kHz, 12.5pF, Q4 IRLML6344TRPBF, Q5 IRLML6344TRPBF, U1 L7985A, U2 L7985A, U3 DS1307ZN+, U4 24AA256-I/SN, U5 CD4050BD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

Commit message: Generate MDP files
Parts:
- 12V, 24V, 3.3V, 5V, 5V/1, BB1, FI1, FI2, FI3, FI4, FI5, FI6, FI7, FI8, GND, GND/1, H1, H2, H3, H4, U$1, U$7, WP: OC_NEWARK (none) -> unknown
- B1: MF KEYSTONE -> KEYSTONE ELECTR; OC_NEWARK (none) -> 66F5622
- BAT: MF MOLEX -> (none); OC_NEWARK (none) -> 98K6552
- C1: MF MURATA -> (none); MPN GRM188R71H471KA01D -> GRM1885C1H471JA01D; OC_NEWARK (none) -> 03AC2702
- C10, C13, C15, C17, C21, C22, C24, C25, C27, C29, C32, C33, C35, C6, C8: MF MULTICOMP -> (none); MPN MC0603B104K250CT -> GRM188R71H104KA93D; OC_NEWARK (none) -> 19X1715
- C11, C2: MF MURATA -> FARNELL; MPN GRM188R71E223KA01D -> GRM188R71H223KA01D; OC_NEWARK (none) -> 38K1672
- C12, C3: MF MURATA -> (none); MPN GRM32ER61C476ME15L -> GRM32ER61C476KE15K; OC_NEWARK (none) -> 96Y9294
- C14, C4: MF MURATA -> (none); MPN GRM32ER71H475KA88L -> GCM32ER71H475KA55L; OC_NEWARK (none) -> 12AC6489
- C19: MF MULTICOMP -> (none); MPN MC0603B562K500CT -> C0603C562J5GACTU; OC_NEWARK (none) -> 79M0848
- C20: MF MURATA -> FARNELL; OC_NEWARK (none) -> 38K1673
- C23, C28, C30, C36, C5: MF AVX (FORMERLY KNOWN AS NICHICON) -> KEMET; MPN F931A475MAA -> T491A475K010AT; OC_NEWARK (none) -> 57K1703
- C26, C46, C7: MF MULTICOMP -> (none); MPN MC0603X475K6R3CT -> GRM188R60J475KE19D; OC_NEWARK (none) -> 03AC2654
- C41: MF MULTICOMP -> (none); MPN MC0603B104K250CT -> GRM188R71H104KA93D; OC_NEWARK 06R4923 -> 19X1715
- C42, C43: MF MULTICOMP -> (none); MPN MC0603B183K160CT -> MC0603N180J500CT
- C9: MF MULTICOMP -> FARNELL; MPN MC0603B331K500CT -> GRM1885C1H331JA01D; OC_NEWARK (none) -> 38K1687
- D1, D2, D3, D4: MF STMICROELECTRONICS -> (none); OC_NEWARK (none) -> 06X0873
- EXP0: OC_NEWARK (none) -> 59J1830
- FB1: MF LAIRD TECHNOLOGIES -> (none); OC_NEWARK (none) -> 66W8861
- FU1: MF KEYSTONE -> (none); OC_NEWARK (none) -> 22M2711
- IC1: MF ATMEL -> (none)
- ISW: MF MOLEX -> (none); OC_NEWARK (none) -> 26M6365
- L1, L4: MF WURTH ELEKTRONIK -> (none)
- LED1: MF MULTICOMP -> (none); OC_NEWARK (none) -> 15R2208
- LED2, LED3, LED4, LED5, LED6, LED7, LED8, LED9: MF MULTICOMP -> (none); OC_NEWARK (none) -> 15R2205
- OK1, OK3: MF VISHAY -> VISHAY/TELEFUNKEN; OC_NEWARK (none) -> 06H1639
- POW: MF PHOENIX CONTACT -> (none)
- Q1: MF ABRACON -> (none); MPN ABS07-32.768KHZ-T -> ABS06-32.768KHZ-T; OC_NEWARK (none) -> 52R7999
- Q4, Q5: MF INFINEON -> (none)
- R1: MF MULTICOMP -> (none); MPN MCMR06X2000FTL -> RC0603FR-07200RL; OC_NEWARK (none) -> 68R0071
- R10, R12, R14, R23, R36, R53, R9: MF MULTICOMP -> (none); MPN MCMR06X1001FTL -> RC0603FR-071KL; OC_NEWARK (none) -> 68R0042
- R11: MF MULTICOMP -> (none); MPN MCWR06X1600FTL -> RC0603FR-07160RL; OC_NEWARK (none) -> 66R2081
- R13, R18, R19, R20, R22, R25, R26, R27, R28, R29, R30, R31, R401, R402, R41: MF MULTICOMP -> (none); MPN MCMR06X4701FTL -> RC0603FR-074K7L; OC_NEWARK (none) -> 68R0092
- R15, R16, R17, R21, R35: MF MULTICOMP -> (none); MPN MCMR06X1501FTL -> RC0603FR-071K5L; OC_NEWARK (none) -> 68R0045
- R2: MF MULTICOMP -> (none); MPN MCMR06X2201FTL -> RC0603FR-072K2L; OC_NEWARK (none) -> 68R0064
- R24: MF MULTICOMP -> (none); MPN MCMR06X3601FTL -> RC0603FR-073K6L; OC_NEWARK (none) -> 68R0080
- R3: MF MULTICOMP -> (none); MPN MCMR06X2700FTL -> RC0603FR-07270RL; OC_NEWARK (none) -> 98K7385
- R32, R38, R40: MF MULTICOMP -> (none); MPN MCMR06X1002FTL -> RC0603FR-0710KL; OC_NEWARK (none) -> 68R0049
- R33: MF MULTICOMP -> (none); MPN MC0063W06031698R -> RC0603FR-07698RL; OC_NEWARK (none) -> 66R2546
- R34, R4: MF MULTICOMP -> (none); MPN MCMR06X5101FTL -> RC0603FR-075K1L; OC_NEWARK (none) -> 68R0101
- R37, R39, R5, R52, R6, R7, R8: MF MULTICOMP -> (none); MPN MCMR06X1000FTL -> RC0603FR-07100RL; OC_NEWARK (none) -> 68R0052
- R42, R51, R57, R58, R59, R60, R62, R63, R64, R65, R66, R67: MF MULTICOMP -> (none); MPN MC0063W060313K3 -> RC0603FR-073K3L; OC_NEWARK (none) -> 68R0079
- R45, R46, R48, R50: MF MULTICOMP -> (none); MPN MCMR06X49R9FTL -> RC0603FR-0749R9L; OC_NEWARK (none) -> 68R0100
- R68: MF MULTICOMP -> (none); MPN MCMR06X3001FTL -> MC0063W060313K01
- R73, R74: MF MULTICOMP -> Multicomp Passives; MPN MCMR06X2200FTL -> MC0063W06031220R
- R75: MF MULTICOMP -> Multicomp Passives; MPN MCMR06X000 PTL -> MC0603WG00000T5E-TC
- R76: MF MULTICOMP -> (none); MPN MCMR06X4701FTL -> RC0603FR-074K7L; OC_NEWARK 58K4608 -> 68R0092
- RL1: MF OMRON ELECTRONIC COMPONENTS -> OMRON COMPONENTS USA; MPN G6L1F5DC -> G6L-1F DC5; OC_NEWARK (none) -> 35K4537
- TH0, TH1, TH2: MF MOLEX -> (none); OC_NEWARK (none) -> 25M1728
- U$4: MF MICREL SEMICONDUCTOR -> (none); MPN KSZ8851SNLI TR -> KSZ8851SNLI-TR
- U1, U2: MF STMICROELECTRONICS -> (none); OC_NEWARK (none) -> unknown
- U3: MF MAXIM INTEGRATED PRODUCTS -> (none); MPN (none) -> DS1307N+; OC_NEWARK (none) -> 73Y1207
- U4: MF MICROCHIP -> (none); OC_NEWARK (none) -> 35M0711
- U5, U6: MF TEXAS INSTRUMENTS -> (none)
- U7: MF NXP -> (none)
- X1: MF TXC -> (none)
