File: ArmazConnectLite/Rev A1/ArmazConnectLite - Rev A1.sch (EAGLE design)
At the start: 17 parts, among them J1 22-05-7028-02, X1 MSTBA3, X8 87832-26

Commit message: Place copyright and board name
Connections:
- new net +24V: X1-1.1
Changed lines of the file:
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@@
 <part name="GND1" library="supply1" deviceset="GND" device=""/>
 <part name="SUPPLY4" library="supply2" deviceset="GND1" device=""/>
+<part name="P+1" library="supply3" deviceset="+24V" device=""/>
 </parts>
 <sheets>
@@
 <instance part="GND1" gate="1" x="50.8" y="154.94" rot="MR0"/>
 <instance part="SUPPLY4" gate="G$1" x="33.02" y="10.16"/>
+<instance part="P+1" gate="1" x="50.8" y="185.42"/>
 </instances>
 <busses>
@@
 </segment>
 </net>
+<net name="+24V" class="0">
+<segment>
+<pinref part="X1" gate="-1" pin="1"/>
+<pinref part="P+1" gate="1" pin="+24V"/>
+<wire x1="43.18" y1="172.72" x2="50.8" y2="172.72" width="0.1524" layer="91"/>
+<wire x1="50.8" y1="172.72" x2="50.8" y2="182.88" width="0.1524" layer="91"/>
+</segment>
+</net>

Commit message: generate gerber and MDP files
Parts:
- removed FI1, FI2, FI3, FI4, FI5, FI6, FI7, FI8: FIDUCIAL1X2, SparkFun:FIDUCIAL1X2
- removed U$1: EXMACHINA-LOGO-NAME, exmachina:EXMACHINA-LOGO-NAME
- removed X8: 87832-26, con-molex:87832-26
- added J4: 22-05-7028-02, con-molex:22-05-7028-02
- added JP1, JP2, JP3, JP4: FIDUCIAL1X2, SparkFun:FIDUCIAL1X2
- added T1: EXMACHINA-LOGO-NAME, exmachina:EXMACHINA-LOGO-NAME
- X1: value MSTBA3 -> 87832-26; device con-phoenix-508:MSTBA3 -> con-molex:87832-26; MF (none) -> MOLEX; MPN (none) -> 87832-2620; OC_FARNELL (none) -> 2313712
- renumbered FAN0 to J2, FAN1 to J3
Connections:
- removed net +24V: X1-1.1
- removed net VDD33A1: X8.24
- new net N$1: X1.24
- net +12V: now also X1.21, X1.22; no longer X8.21, X8.22
- net +5V: now also X1.1, X1.2; no longer X8.1, X8.2
- net +5V/1: now also J4-1.S, X1.23; no longer J1-1.S, X8.23
- net ESW0: now also X1.5; no longer X8.5
- net ESW1: now also X1.6; no longer X8.6
- net ESW2: now also X1.7; no longer X8.7
- net ESW3: now also X1.8; no longer X8.8
- net ESW4: now also J1-1.S, X1.15; no longer X1-2.1, X8.15
- net ESW5: now also X1.13; no longer X8.13
- net ESW6: now also X1.14; no longer X8.14
- net FAN0_GND: now also X1.19; no longer X8.19
- net FAN1_GND: now also X1.20; no longer X8.20
- net GND: now also J1-2.S, X1.3, X1.4; no longer X1-3.1, X8.3, X8.4
- net GND1: now also J4-2.S, X1.25, X1.26; no longer J1-2.S, X8.25, X8.26
- net OUT0: now also X1.16; no longer X8.16
- net OUT1: now also X1.17; no longer X8.17
- net OUT2: now also X1.18; no longer X8.18
- net UART4_RXD: now also X1.11; no longer X8.11
- net UART4_TXD: now also X1.12; no longer X8.12
- net UART5_RXD: now also X1.9; no longer X8.9
- net UART5_TXD: now also X1.10; no longer X8.10
Other:
- moved on the sheet: J1-1, J1-2, MP1, MP2
