File: ArmazRelay/Rev A1/ArmazRelay - RevA1.sch (EAGLE design)
At the start: 5 parts, among them J1 22-05-7028-02, J2 MSTBA3, K1 MY2

Commit message: Update board
Parts:
- added CC1: CC-BY-NC-SA, cc-by-sa:CC-BY-NC-SA
- added T1: EXMACHINA-LOGO-NAME, exmachina:EXMACHINA-LOGO-NAME
Connections:
- new net +24V: J2-1.1, K1G$2.C
- new net GND: J1-2.S, J2-3.1, K1G$1.COIL2
- new net SIG_IN: J2-2.1, K1G$1.COIL1
- new net SIG_OUT: J1-1.S, K1G$2.NC
Other:
- moved on the sheet: J2-1, J2-2, J2-3, K1
Changed lines of the file:
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@@
 <part name="J2" library="con-phoenix-508" deviceset="MSTBA3" device=""/>
 <part name="K1" library="rel-omron" deviceset="MY2" device=""/>
+<part name="P+1" library="supply3" deviceset="+24V" device=""/>
+<part name="GND1" library="supply3" deviceset="GND" device=""/>
+<part name="GND2" library="supply3" deviceset="GND" device=""/>
+<part name="GND3" library="supply3" deviceset="GND" device=""/>
+<part name="P+2" library="supply3" deviceset="+24V" device=""/>
+<part name="CC1" library="cc-by-sa" deviceset="CC-BY-NC-SA" device=""/>
+<part name="T1" library="exmachina" deviceset="EXMACHINA-LOGO" device="-NAME"/>
 </parts>
 <sheets>
@@
 <instance part="J1" gate="-1" x="24.13" y="236.22" rot="MR0"/>
 <instance part="J1" gate="-2" x="24.13" y="231.14" rot="MR0"/>
-<instance part="J2" gate="-1" x="24.13" y="217.17"/>
-<instance part="J2" gate="-2" x="24.13" y="212.09"/>
-<instance part="J2" gate="-3" x="24.13" y="207.01"/>
-<instance part="K1" gate="G$2" x="168.91" y="227.33" rot="R90"/>
-<instance part="K1" gate="G$3" x="168.91" y="203.2" rot="R90"/>
+<instance part="J2" gate="-1" x="24.13" y="213.36"/>
+<instance part="J2" gate="-2" x="24.13" y="208.28"/>
+<instance part="J2" gate="-3" x="24.13" y="203.2"/>
+<instance part="K1" gate="G$2" x="162.56" y="217.17" rot="MR90"/>
 <instance part="K1" gate="G$1" x="140.97" y="217.17"/>
+<instance part="P+1" gate="1" x="34.29" y="219.71"/>
+<instance part="GND1" gate="1" x="34.29" y="198.12"/>
+<instance part="GND2" gate="1" x="34.29" y="227.33"/>
+<instance part="GND3" gate="1" x="140.97" y="205.74"/>
+<instance part="P+2" gate="1" x="157.48" y="231.14"/>
+<instance part="CC1" gate="G$1" x="303.53" y="8.89"/>
+<instance part="T1" gate="G$1" x="311.15" y="19.05"/>
 </instances>
 <busses>
 </busses>
 <nets>
+<net name="+24V" class="0">
+<segment>
+<pinref part="J2" gate="-1" pin="1"/>
+<pinref part="P+1" gate="1" pin="+24V"/>
+<wire x1="29.21" y1="213.36" x2="34.29" y2="213.36" width="0.1524" layer="91"/>
+<wire x1="34.29" y1="213.36" x2="34.29" y2="217.17" width="0.1524" layer="91"/>
+</segment>
+<segment>
+<pinref part="K1" gate="G$2" pin="C"/>
+<pinref part="P+2" gate="1" pin="+24V"/>
+<wire x1="160.02" y1="217.17" x2="157.48" y2="217.17" width="0.1524" layer="91"/>
+<wire x1="157.48" y1="217.17" x2="157.48" y2="228.6" width="0.1524" layer="91"/>
+</segment>
+</net>
+<net name="GND" class="0">
+<segment>
+<pinref part="J2" gate="-3" pin="1"/>
+<pinref part="GND1" gate="1" pin="GND"/>
+<wire x1="29.21" y1="203.2" x2="34.29" y2="203.2" width="0.1524" layer="91"/>
+<wire x1="34.29" y1="203.2" x2="34.29" y2="200.66" width="0.1524" layer="91"/>
+</segment>
+<segment>
+<pinref part="J1" gate="-2" pin="S"/>
+<pinref part="GND2" gate="1" pin="GND"/>
+<wire x1="26.67" y1="231.14" x2="34.29" y2="231.14" width="0.1524" layer="91"/>
+<wire x1="34.29" y1="231.14" x2="34.29" y2="229.87" width="0.1524" layer="91"/>
+</segment>
+<segment>
+<pinref part="K1" gate="G$1" pin="COIL2"/>
+<pinref part="GND3" gate="1" pin="GND"/>
+<wire x1="140.97" y1="212.09" x2="140.97" y2="208.28" width="0.1524" layer="91"/>
+</segment>
+</net>
+<net name="SIG_IN" class="0">
+<segment>
+<pinref part="J2" gate="-2" pin="1"/>
+<wire x1="29.21" y1="208.28" x2="36.83" y2="208.28" width="0.1524" layer="91"/>
+<label x="36.83" y="208.28" size="1.27" layer="95" xref="yes"/>
+</segment>
+<segment>
+<wire x1="133.35" y1="226.06" x2="140.97" y2="226.06" width="0.1524" layer="91"/>
+<pinref part="K1" gate="G$1" pin="COIL1"/>
+<wire x1="140.97" y1="226.06" x2="140.97" y2="222.25" width="0.1524" layer="91"/>
+<label x="133.35" y="226.06" size="1.27" layer="95" rot="R180" xref="yes"/>
+</segment>
+</net>
+<net name="SIG_OUT" class="0">
+<segment>
+<pinref part="J1" gate="-1" pin="S"/>
+<wire x1="26.67" y1="236.22" x2="36.83" y2="236.22" width="0.1524" layer="91"/>
+<label x="36.83" y="236.22" size="1.27" layer="95" xref="yes"/>
+</segment>
+<segment>
+<wire x1="167.64" y1="209.55" x2="177.8" y2="209.55" width="0.1524" layer="91"/>
+<pinref part="K1" gate="G$2" pin="NC"/>
+<wire x1="167.64" y1="209.55" x2="167.64" y2="212.09" width="0.1524" layer="91"/>
+<label x="177.8" y="209.55" size="1.27" layer="95" xref="yes"/>
+</segment>
+</net>
 </nets>
 </sheet>

Commit message: Add power connector and NC output
Parts:
- added J3: MSTBA2, con-phoenix-508:MSTBA2
- J1: value 22-05-7028-02 -> 22-05-7038-03; device con-molex:22-05-7028-02 -> con-molex:22-05-7038-03
Connections:
- removed net SIG_OUT: J1-1.S, K1G$2.NC
- new net SIG_NC: J1-1.S, K1G$2.NO
- new net SIG_NO: J1-2.S, K1G$2.NC
- net +24V: now also J3-1.1
- net GND: now also J1-3.S, J3-2.1; no longer J1-2.S
Other:
- moved on the sheet: H1, J1-1, J1-2, J2-1, J2-2, J2-3, K1

Commit message: Final review of ArmazRelay board
- Add second output
- Change trace width to 32mil
- Add silkscreen labels
- Enlarge pad rings on the relay
Parts:
- added J4: 22-05-7038-03, con-molex:22-05-7038-03
- H1, H2: value MOUNT-HOLE3.0 -> MOUNT-PAD3,0; device holes:MOUNT-HOLE3.0 -> holes:MOUNT-PAD3,0
- J1: value 22-05-7038-03 -> MSTBA2; device con-molex:22-05-7038-03 -> con-phoenix-508:MSTBA2
- J3: value MSTBA2 -> 22-05-7038-03; device con-phoenix-508:MSTBA2 -> con-molex:22-05-7038-03
Connections:
- removed net SIG_NC: J1-1.S, K1G$2.NO
- removed net SIG_NO: J1-2.S, K1G$2.NC
- new net SIG1_NC: J4-1.S, K1G$2.NO
- new net SIG1_NO: J4-2.S, K1G$2.NC
- new net SIG2_NC: J3-1.S, K1G$3.NO
- new net SIG2_NO: J3-2.S, K1G$3.NC
- net +24V: now also J1-1.1, K1G$3.C; no longer J3-1.1
- net GND: now also J1-2.1, J3-3.S, J4-3.S; no longer J1-3.S, J3-2.1
Changed lines of the file:
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@@
 </variantdefs>
 <classes>
-<class number="0" name="default" width="0" drill="0">
+<class number="0" name="default" width="0.8128" drill="0">
 </class>
 </classes>
 <parts>
 <part name="FRAME1" library="frames" deviceset="A3L-LOC" device=""/>
-<part name="H1" library="holes" deviceset="MOUNT-HOLE" device="3.0"/>
-<part name="H2" library="holes" deviceset="MOUNT-HOLE" device="3.0"/>
+<part name="H1" library="holes" deviceset="MOUNT-PAD" device="3,0"/>
+<part name="H2" library="holes" deviceset="MOUNT-PAD" device="3,0"/>
 <part name="J2" library="con-phoenix-508" deviceset="MSTBA3" device=""/>
 <part name="K1" library="rel-omron" deviceset="MY2" device=""/>
@@
 <part name="CC1" library="cc-by-sa" deviceset="CC-BY-NC-SA" device=""/>
 <part name="T1" library="exmachina" deviceset="EXMACHINA-LOGO" device="-NAME"/>
-<part name="J3" library="con-phoenix-508" deviceset="MSTBA2" device=""/>
+<part name="J1" library="con-phoenix-508" deviceset="MSTBA2" device=""/>
 <part name="P+3" library="supply3" deviceset="+24V" device=""/>
 <part name="GND4" library="supply3" deviceset="GND" device=""/>
-<part name="J1" library="con-molex" deviceset="22-?-03" device="05-7038"/>
+<part name="J4" library="con-molex" deviceset="22-?-03" device="05-7038"/>
+<part name="J3" library="con-molex" deviceset="22-?-03" device="05-7038"/>
+<part name="GND5" library="supply3" deviceset="GND" device=""/>
 </parts>
 <sheets>
@@
 <instances>
 <instance part="FRAME1" gate="G$1" x="0" y="0"/>
-<instance part="H1" gate="G$1" x="360.68" y="30.48"/>
-<instance part="H2" gate="G$1" x="335.28" y="30.48"/>
+<instance part="H1" gate="1" x="360.68" y="30.48"/>
+<instance part="H2" gate="1" x="335.28" y="30.48"/>
 <instance part="J2" gate="-1" x="25.4" y="213.36"/>
 <instance part="J2" gate="-2" x="25.4" y="208.28"/>
@@
 <instance part="CC1" gate="G$1" x="304.8" y="10.16"/>
 <instance part="T1" gate="G$1" x="312.42" y="20.32"/>
-<instance part="J3" gate="-1" x="22.86" y="175.26"/>
-<instance part="J3" gate="-2" x="22.86" y="170.18"/>
+<instance part="J1" gate="-1" x="22.86" y="175.26"/>
+<instance part="J1" gate="-2" x="22.86" y="170.18"/>
 <instance part="P+3" gate="1" x="35.56" y="182.88"/>
 <instance part="GND4" gate="1" x="35.56" y="165.1"/>
-<instance part="J1" gate="-1" x="25.4" y="241.3" rot="MR0"/>
-<instance part="J1" gate="-2" x="25.4" y="236.22" rot="MR0"/>
-<instance part="J1" gate="-3" x="25.4" y="231.14" rot="MR0"/>
+<instance part="J4" gate="-1" x="25.4" y="241.3" rot="MR0"/>
+<instance part="J4" gate="-2" x="25.4" y="236.22" rot="MR0"/>
+<instance part="J4" gate="-3" x="25.4" y="231.14" rot="MR0"/>
+<instance part="K1" gate="G$3" x="162.56" y="195.58" rot="MR90"/>
+<instance part="J3" gate="-1" x="73.66" y="241.3" rot="MR0"/>
+<instance part="J3" gate="-2" x="73.66" y="236.22" rot="MR0"/>
+<instance part="J3" gate="-3" x="73.66" y="231.14" rot="MR0"/>
+<instance part="GND5" gate="1" x="86.36" y="228.6"/>
 </instances>
 <busses>
@@
 <wire x1="160.02" y1="218.44" x2="157.48" y2="218.44" width="0.1524" layer="91"/>
 <wire x1="157.48" y1="218.44" x2="157.48" y2="228.6" width="0.1524" layer="91"/>
+<pinref part="K1" gate="G$3" pin="C"/>
+<wire x1="160.02" y1="195.58" x2="157.48" y2="195.58" width="0.1524" layer="91"/>
+<wire x1="157.48" y1="195.58" x2="157.48" y2="218.44" width="0.1524" layer="91"/>
+<junction x="157.48" y="218.44"/>
 </segment>
 <segment>
-<pinref part="J3" gate="-1" pin="1"/>
+<pinref part="J1" gate="-1" pin="1"/>
 <pinref part="P+3" gate="1" pin="+24V"/>
 <wire x1="27.94" y1="175.26" x2="35.56" y2="175.26" width="0.1524" layer="91"/>
@@
 <pinref part="GND2" gate="1" pin="GND"/>
 <wire x1="27.94" y1="231.14" x2="35.56" y2="231.14" width="0.1524" layer="91"/>
-<pinref part="J1" gate="-3" pin="S"/>
+<pinref part="J4" gate="-3" pin="S"/>
 </segment>
 <segment>
@@
 </segment>
 <segment>
-<pinref part="J3" gate="-2" pin="1"/>
+<pinref part="J1" gate="-2" pin="1"/>
 <pinref part="GND4" gate="1" pin="GND"/>
 <wire x1="27.94" y1="170.18" x2="35.56" y2="170.18" width="0.1524" layer="91"/>
 <wire x1="35.56" y1="170.18" x2="35.56" y2="167.64" width="0.1524" layer="91"/>
+</segment>
+<segment>
+<pinref part="J3" gate="-3" pin="S"/>
+<wire x1="76.2" y1="231.14" x2="86.36" y2="231.14" width="0.1524" layer="91"/>
+<pinref part="GND5" gate="1" pin="GND"/>
 </segment>
 </net>
@@
 </segment>
 </net>
-<net name="SIG_NO" class="0">
+<net name="SIG1_NO" class="0">
 <segment>
 <wire x1="27.94" y1="236.22" x2="38.1" y2="236.22" width="0.1524" layer="91"/>
 <label x="38.1" y="236.22" size="1.27" layer="95" xref="yes"/>
-<pinref part="J1" gate="-2" pin="S"/>
+<pinref part="J4" gate="-2" pin="S"/>
 </segment>
 <segment>
@@
 </segment>
 </net>
-<net name="SIG_NC" class="0">
+<net name="SIG1_NC" class="0">
 <segment>
-<pinref part="J1" gate="-1" pin="S"/>
+<pinref part="J4" gate="-1" pin="S"/>
 <wire x1="27.94" y1="241.3" x2="38.1" y2="241.3" width="0.1524" layer="91"/>
 <label x="38.1" y="241.3" size="1.27" layer="95" xref="yes"/>
@@
 <pinref part="K1" gate="G$2" pin="NO"/>
 <wire x1="167.64" y1="223.52" x2="167.64" y2="226.06" width="0.1524" layer="91"/>
+<label x="177.8" y="226.06" size="1.27" layer="95" xref="yes"/>
 <wire x1="167.64" y1="226.06" x2="177.8" y2="226.06" width="0.1524" layer="91"/>
-<label x="177.8" y="226.06" size="1.27" layer="95" xref="yes"/>
 </segment>
 </net>
+<net name="SIG2_NC" class="0">
+<segment>
+<pinref part="K1" gate="G$3" pin="NO"/>
+<wire x1="167.64" y1="200.66" x2="167.64" y2="203.2" width="0.1524" layer="91"/>
+<wire x1="167.64" y1="203.2" x2="177.8" y2="203.2" width="0.1524" layer="91"/>
+<label x="177.8" y="203.2" size="1.27" layer="95" xref="yes"/>
+</segment>
+<segment>
+<pinref part="J3" gate="-1" pin="S"/>
+<wire x1="76.2" y1="241.3" x2="86.36" y2="241.3" width="0.1524" layer="91"/>
+<label x="86.36" y="241.3" size="1.27" layer="95" xref="yes"/>
+</segment>
+</net>
+<net name="SIG2_NO" class="0">
+<segment>
+<pinref part="K1" gate="G$3" pin="NC"/>
+<wire x1="167.64" y1="190.5" x2="167.64" y2="187.96" width="0.1524" layer="91"/>
+<wire x1="167.64" y1="187.96" x2="177.8" y2="187.96" width="0.1524" layer="91"/>
+<label x="177.8" y="187.96" size="1.27" layer="95" xref="yes"/>
+</segment>
+<segment>
+<pinref part="J3" gate="-2" pin="S"/>
+<wire x1="76.2" y1="236.22" x2="86.36" y2="236.22" width="0.1524" layer="91"/>
+<label x="86.36" y="236.22" size="1.27" layer="95" xref="yes"/>
+</segment>
+</net>
