File: ArmazRelay/Rev A2/ArmazRelay - Rev A2.brd (EAGLE design)
At the start: 70 x 30 mm, 10 parts, among them J1 MSTBA2, J2 MSTBA3, J3 22-05-7038-03, J4 22-05-7038-03, K1 MY2, T1 EXMACHINA-LOGO-NAME

Commit message: Update relay package and add polarity on relay coil
Routing:
- net SIG2_NC: track 26.0 -> 28.4 mm
- net SIG1_NO: track 20.8 -> 22.4 mm
- net SIG2_NO: track 20.9 -> 22.4 mm
- net SIG_IN: track 31.3 -> 29.8 mm
- net SIG1_NC: track 27.7 -> 28.3 mm
Other:
- board text added: "EXM Relay One RevA2"
- board text removed: "ArmazRelay RevA2"
Changed lines of the file:
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@@
 <setting verticaltext="up"/>
 </settings>
-<grid distance="1" unitdist="mm" unit="mil" style="lines" multiple="1" display="no" altdistance="0.1" altunitdist="mm" altunit="mm"/>
+<grid distance="1" unitdist="mm" unit="mm" style="lines" multiple="1" display="no" altdistance="0.1" altunitdist="mm" altunit="mm"/>
 <layers>
 <layer number="1" name="Top" color="4" fill="1" visible="yes" active="yes"/>
@@
 <layer number="46" name="Milling" color="3" fill="1" visible="no" active="yes"/>
 <layer number="47" name="Measures" color="7" fill="1" visible="no" active="yes"/>
-<layer number="48" name="Document" color="7" fill="1" visible="no" active="yes"/>
+<layer number="48" name="Document" color="7" fill="1" visible="yes" active="yes"/>
 <layer number="49" name="Reference" color="7" fill="1" visible="no" active="yes"/>
 <layer number="50" name="dxf" color="7" fill="1" visible="no" active="yes"/>
@@
 <wire x1="67" y1="30" x2="3" y2="30" width="0" layer="20"/>
 <wire x1="3" y1="30" x2="0" y2="27" width="0" layer="20" curve="90"/>
-<text x="56.3" y="26.2" size="1.016" layer="21" align="top-left">ArmazRelay
+<text x="56.3" y="26.2" size="1.016" layer="21" align="top-left">EXM Relay One
 RevA2</text>
 <text x="10.3" y="26.2" size="1.016" layer="21" align="center-left">+24V</text>
@@
 <signal name="GND">
 <contactref element="J2" pad="3"/>
-<contactref element="K1" pad="13"/>
 <polygon width="0.8128" layer="16" isolate="0.3048">
 <vertex x="-13" y="43"/>
@@
 <contactref element="J4" pad="3"/>
 <contactref element="J3" pad="3"/>
+<contactref element="K1" pad="13"/>
 </signal>
 <signal name="SIG_IN">
 <contactref element="J2" pad="2"/>
-<contactref element="K1" pad="14"/>
 <wire x1="7.08" y1="9" x2="20" y2="9" width="0.8128" layer="1"/>
 <wire x1="20" y1="9" x2="22" y2="11" width="0.8128" layer="1"/>
 <wire x1="22" y1="11" x2="22" y2="19" width="0.8128" layer="1"/>
-<wire x1="22" y1="19" x2="24.5" y2="21.5" width="0.8128" layer="1"/>
-<wire x1="24.5" y1="21.5" x2="28.5" y2="21.5" width="0.8128" layer="1"/>
+<wire x1="22" y1="19" x2="24.605" y2="21.605" width="0.8128" layer="1"/>
+<contactref element="K1" pad="14"/>
+<wire x1="24.605" y1="21.605" x2="26.925" y2="21.605" width="0.8128" layer="1"/>
 </signal>
 <signal name="SIG1_NO">
 <contactref element="K1" pad="4"/>
 <contactref element="J4" pad="2"/>
-<wire x1="45.25" y1="21.5" x2="56.5" y2="21.5" width="0.8128" layer="1"/>
-<wire x1="56.5" y1="21.5" x2="59" y2="19" width="0.8128" layer="1"/>
+<wire x1="56.395" y1="21.605" x2="59" y2="19" width="0.8128" layer="1"/>
 <wire x1="59" y1="19" x2="65" y2="19" width="0.8128" layer="1"/>
+<wire x1="56.395" y1="21.605" x2="43.675" y2="21.605" width="0.8128" layer="1"/>
 </signal>
 <signal name="SIG1_NC">
 <contactref element="J4" pad="1"/>
 <contactref element="K1" pad="8"/>
-<wire x1="41.15" y1="21.5" x2="41.15" y2="23.15" width="0.8128" layer="1"/>
-<wire x1="41.15" y1="23.15" x2="43" y2="25" width="0.8128" layer="1"/>
-<wire x1="43" y1="25" x2="58" y2="25" width="0.8128" layer="1"/>
+<wire x1="42.97" y1="25" x2="58" y2="25" width="0.8128" layer="1"/>
 <wire x1="58" y1="25" x2="61.46" y2="21.54" width="0.8128" layer="1"/>
 <wire x1="61.46" y1="21.54" x2="65" y2="21.54" width="0.8128" layer="1"/>
+<wire x1="42.97" y1="25" x2="39.575" y2="21.605" width="0.8128" layer="1"/>
 </signal>
 <signal name="SIG2_NC">
 <contactref element="K1" pad="5"/>
 <contactref element="J3" pad="1"/>
-<wire x1="65" y1="13.54" x2="61.54" y2="13.54" width="0.8128" layer="1"/>
-<wire x1="61.54" y1="13.54" x2="58" y2="10" width="0.8128" layer="1"/>
-<wire x1="58" y1="10" x2="42.85" y2="10" width="0.8128" layer="1"/>
-<wire x1="42.85" y1="10" x2="41.15" y2="8.3" width="0.8128" layer="1"/>
+<wire x1="65" y1="13.54" x2="60.54" y2="13.54" width="0.8128" layer="1"/>
+<wire x1="60.54" y1="13.54" x2="58" y2="11" width="0.8128" layer="1"/>
+<wire x1="58" y1="11" x2="52" y2="11" width="0.8128" layer="1"/>
+<wire x1="52" y1="11" x2="51" y2="12" width="0.8128" layer="1"/>
+<wire x1="51" y1="12" x2="43.17" y2="12" width="0.8128" layer="1"/>
+<wire x1="43.17" y1="12" x2="39.575" y2="8.405" width="0.8128" layer="1"/>
 </signal>
 <signal name="SIG2_NO">
 <contactref element="K1" pad="1"/>
 <contactref element="J3" pad="2"/>
-<wire x1="45.25" y1="8.3" x2="59.3" y2="8.3" width="0.8128" layer="1"/>
-<wire x1="59.3" y1="8.3" x2="62" y2="11" width="0.8128" layer="1"/>
+<wire x1="59.405" y1="8.405" x2="62" y2="11" width="0.8128" layer="1"/>
 <wire x1="62" y1="11" x2="65" y2="11" width="0.8128" layer="1"/>
+<wire x1="59.405" y1="8.405" x2="43.675" y2="8.405" width="0.8128" layer="1"/>
 </signal>
 </signals>
